Commit message: This works but is using the urdf not the xacro.

File: urdf/robotiq_hande.urdf.xacro (robot description, xacro)
@@ -1,6 +1,26 @@
 <?xml version="1.0"?>
 <robot xmlns:xacro="http://ros.org/wiki/xacro">
-  <xacro:macro name="robotiq_hande"  params="prefix MAC">
-    <link name="${prefix}robotiq_hande_base_link">
+  <xacro:arg name="jaw_xacro" default="standard" />
+  <xacro:arg name="use_fake_hardware" default="false" />
+  <xacro:property name="jaw_xacro_prop" value="$(arg jaw_xacro)" />
+  <!--<xacro:include filename="$(find robotiq_hande_description)/urdf/robotiq_hande_transmission.xacro"/>
+  <xacro:include filename="$(find robotiq_hande_description)/urdf/robotiq_hande_ros2_control.xacro"/>-->
+  <xacro:macro name="robotiq_hande" params="
+    name
+    prefix
+    parent
+    *origin">
+    <material name="${prefix}_dark_gray">
+      <color rgba="0.2 0.2 0.2 1"/>
+    </material>
+    <material name="${prefix}_black">
+      <color rgba="0 0 0 1"/>
+    </material>
+    <joint name="${prefix}gripper_base_joint" type="fixed">
+      <parent link="${parent}"/>
+      <child link="${prefix}gripper_base_link"/>
+      <xacro:insert_block name="origin"/>
+    </joint>
+    <link name="${prefix}gripper_base_link">
       <inertial>
         <origin xyz="0 0 0.04607" rpy="0 0 0" />
@@ -13,7 +33,5 @@
           <mesh filename="package://robotiq_hande_description/meshes/hand-e.dae" scale="0.001 0.001 0.001"/>
         </geometry>
-        <material name="Gazebo/Black">
-          <color rgba="0.1 0.1 0.1 1" />
-        </material>
+        <material name="${prefix}_black"/>
       </visual>
       <collision>
@@ -24,9 +42,25 @@
       </collision>
     </link>
-    <gazebo reference="${prefix}robotiq_hande_base_link">
-      <material>Gazebo/Black</material>
-      <selfCollide>True</selfCollide>
-    </gazebo>
-    <link name="${prefix}left_finger">
+    <link name="${prefix}finger_1_link">
+      <inertial>
+        <origin rpy="0 0 0" xyz="-0.02262 0.00759 0.00738"/>
+        <mass value="0.03804"/>
+        <inertia ixx="13567E-9" ixy="1849E-9" ixz="-3622E-9" iyy="15784E-9" iyz="-3616E-9" izz="7478E-9"/>
+      </inertial>
+      <visual>
+        <origin rpy="0 0 0" xyz="0 0 0"/>
+        <geometry>
+          <mesh filename="package://robotiq_hande_description/meshes/finger_2.dae" scale="0.001 0.001 0.001"/>
+        </geometry>
+        <material name="${prefix}_dark_gray"/>
+      </visual>
+      <collision>
+        <origin rpy="0 0 0" xyz="0 0 0"/>
+        <geometry>
+          <mesh filename="package://robotiq_hande_description/meshes/finger_2.dae" scale="0.001 0.001 0.001"/>
+        </geometry>
+      </collision>
+    </link>
+    <link name="${prefix}finger_2_link">
       <inertial>
         <origin rpy="0 0 0" xyz="0.02262 -0.00759 0.00738"/>
@@ -39,7 +73,5 @@
           <mesh filename="package://robotiq_hande_description/meshes/finger_1.dae" scale="0.001 0.001 0.001"/>
         </geometry>
-        <material name="Gazebo/Grey">
-          <color rgba="0.1 0.1 0.1 1"/>
-        </material>
+        <material name="${prefix}_dark_gray"/>
       </visual>
       <collision>
@@ -50,60 +82,19 @@
       </collision>
     </link>
-    <gazebo reference="${prefix}left_finger">
-      <material>Gazebo/Grey</material>
-      <selfCollide>True</selfCollide>
-    </gazebo>
-    <link name="${prefix}right_finger">
-      <inertial>
-        <origin rpy="0 0 0" xyz="-0.02262 0.00759 0.00738"/>
-        <mass value="0.03804"/>
-        <inertia ixx="13567E-9" ixy="1849E-9" ixz="-3622E-9" iyy="15784E-9" iyz="-3616E-9" izz="7478E-9"/>
-      </inertial>
-      <visual>
-        <origin rpy="0 0 0" xyz="0 0 0"/>
-        <geometry>
-          <mesh filename="package://robotiq_hande_description/meshes/finger_2.dae" scale="0.001 0.001 0.001"/>
-        </geometry>
-        <material name="Gazebo/Grey">
-          <color rgba="0.1 0.1 0.1 1"/>
-        </material>
-      </visual>
-      <collision>
-        <origin rpy="0 0 0" xyz="0 0 0"/>
-        <geometry>
-          <mesh filename="package://robotiq_hande_description/meshes/finger_2.dae" scale="0.001 0.001 0.001"/>
-        </geometry>
-      </collision>
-    </link>
-    <gazebo reference="${prefix}right_finger">
-      <material>Gazebo/Grey</material>
-      <selfCollide>True</selfCollide>
-    </gazebo>
-    <joint name="${prefix}joint_finger" type="prismatic">
+    <joint name="${prefix}finger_1_joint" type="prismatic">
       <origin rpy="0 0 0" xyz="0 0 0.099"/>
-      <parent link="${prefix}robotiq_hande_base_link"/>
-      <child link="${prefix}left_finger"/>
-      <axis xyz="-1 0 0"/>
-      <limit effort="130" lower="0" upper="0.025" velocity="0.15"/>
-    </joint>
-    <joint name="robotiq_hande_base_to_${prefix}right_finger" type="prismatic">
-      <origin rpy="0 0 0" xyz="0 0 0.099"/>
-      <parent link="${prefix}robotiq_hande_base_link"/>
-      <child link="${prefix}right_finger"/>
+      <parent link="${prefix}gripper_base_link"/>
+      <child link="${prefix}finger_1_link"/>
       <axis xyz="1 0 0"/>
       <limit effort="130" lower="0" upper="0.025" velocity="0.15"/>
       <mimic joint="${prefix}joint_finger" multiplier="1" offset="0"/>
     </joint>
-    <gazebo>
-      <plugin filename="librobotiq_gazebo_plugin.so" name="hrim_actuator_gripper${MAC}">
-        <kp>500</kp>
-        <ki>3</ki>
-        <kd>9</kd>
-        <min_velocity>20</min_velocity>
-        <max_velocity>150</max_velocity>
-        <joint>${prefix}joint_finger</joint>
-        <joint>robotiq_hande_base_to_${prefix}right_finger</joint>
-      </plugin>
-    </gazebo>
+    <joint name="${prefix}finger_2_joint" type="prismatic">
+      <origin rpy="0 0 0" xyz="0 0 0.099"/>
+      <parent link="${prefix}gripper_base_link"/>
+      <child link="${prefix}finger_2_link"/>
+      <axis xyz="-1 0 0"/>
+      <limit effort="130" lower="0" upper="0.025" velocity="0.15"/>
+    </joint>
   </xacro:macro>
 </robot>

File: urdf/robotiq_hande_world.urdf.xacro (robot description, xacro)
@@ -3,5 +3,5 @@
   <!-- robotiq_hande_gripper -->
   <xacro:include filename="$(find robotiq_hande_description)/urdf/robotiq_hande.urdf.xacro" />
-  <xacro:robotiq_hande prefix="hande_" MAC="_000000000004"/>
+  <xacro:robotiq_hande prefix="hande_" parent=""/>
   <link name="world" />
   <joint name="world_to_robotiq_adapter" type="fixed">

Commit message: Updates and upgrades. Working with the xacro now. No ROS2 control.4

File: urdf/robotiq_hande.urdf.xacro (robot description, xacro)
@@ -11,8 +11,8 @@
     parent
     *origin">
-    <material name="${prefix}_dark_gray">
+    <material name="${prefix}dark_gray">
       <color rgba="0.2 0.2 0.2 1"/>
     </material>
-    <material name="${prefix}_black">
+    <material name="${prefix}black">
       <color rgba="0 0 0 1"/>
     </material>
@@ -33,5 +33,5 @@
           <mesh filename="package://robotiq_hande_description/meshes/hand-e.dae" scale="0.001 0.001 0.001"/>
         </geometry>
-        <material name="${prefix}_black"/>
+        <material name="${prefix}black"/>
       </visual>
       <collision>
@@ -53,5 +53,5 @@
           <mesh filename="package://robotiq_hande_description/meshes/finger_2.dae" scale="0.001 0.001 0.001"/>
         </geometry>
-        <material name="${prefix}_dark_gray"/>
+        <material name="${prefix}dark_gray"/>
       </visual>
       <collision>
@@ -73,5 +73,5 @@
           <mesh filename="package://robotiq_hande_description/meshes/finger_1.dae" scale="0.001 0.001 0.001"/>
         </geometry>
-        <material name="${prefix}_dark_gray"/>
+        <material name="${prefix}dark_gray"/>
       </visual>
       <collision>
@@ -88,5 +88,4 @@
       <axis xyz="1 0 0"/>
       <limit effort="130" lower="0" upper="0.025" velocity="0.15"/>
-      <mimic joint="${prefix}joint_finger" multiplier="1" offset="0"/>
     </joint>
     <joint name="${prefix}finger_2_joint" type="prismatic">
@@ -96,4 +95,5 @@
       <axis xyz="-1 0 0"/>
       <limit effort="130" lower="0" upper="0.025" velocity="0.15"/>
+      <mimic joint="${prefix}finger_1_joint" multiplier="1" offset="0"/>
     </joint>
   </xacro:macro>

File: urdf/robotiq_hande_ros2_control.xacro (robot description, xacro)
@@ -9,8 +9,8 @@
     </hardware>
     <joint name="${prefix}finger_1_joint">
-      <param name="initial_position">0.00075</param>
+      <param name="initial_position">0.00</param>
       <command_interface name="position">
-        <param name="min">0.00075</param>
-        <param name="max">0.04</param>
+        <param name="min">0.00</param>
+        <param name="max">0.05</param>
       </command_interface>
       <state_interface name="position"/>

Commit message: Added grasp, push, and finger tip frame.

File: urdf/robotiq_hande.urdf.xacro (robot description, xacro)
@@ -97,4 +97,60 @@
       <mimic joint="${prefix}finger_1_joint" multiplier="1" offset="0"/>
     </joint>
+    <link name="${prefix}grasp_frame">
+      <visual>
+        <geometry>
+          <sphere radius="0.007"/>
+        </geometry>
+        <material name="${prefix}_green">
+          <color rgba="0 1.0 0 1.0"/>
+        </material>
+      </visual>
+    </link>
+    <joint name="${prefix}grasp_frame_joint" type="fixed">
+      <parent link="${prefix}gripper_base_link"/>
+      <child link="${prefix}grasp_frame"/>
+      <xacro:if value="${jaw_xacro_prop == 'standard'}" >
+        <origin xyz="0.0 0.0 0.135" rpy="0 0 0"/>
+      </xacro:if>
+    </joint>
+    <link name="${prefix}push_frame">
+      <visual>
+        <geometry>
+          <box size="0.014 0.014 0.014"/>
+        </geometry>
+        <material name="${prefix}_red">
+          <color rgba="1.0 0 0 1.0"/>
+        </material>
+      </visual>
+    </link>
+    <joint name="${prefix}push_frame_joint" type="fixed">
+      <parent link="${prefix}gripper_base_link"/>
+      <child link="${prefix}push_frame"/>
+      <xacro:if value="${jaw_xacro_prop == 'standard'}" >
+        <origin xyz="0.0 0.0 0.147" rpy="0 0 0"/>
+      </xacro:if>
+    </joint>
+    <!--Calibration frame-->
+    <link name="${prefix}gripper_calibration_link"/>
+    <joint name="${prefix}gripper_finger_base_joint" type="fixed">
+      <parent link="${prefix}gripper_base_link"/>
+      <child link="${prefix}gripper_calibration_link"/>
+      <origin xyz="0.0 0.0 0.099" rpy="0 0 0"/>
+    </joint>
+    <!--Fingertip frames-->
+    <link name="${prefix}finger_1_fingertip_link"/>
+    <joint name="${prefix}finger_1_fingertip_joint" type="fixed">
+      <parent link="${prefix}finger_1_link"/>
+      <child link="${prefix}finger_1_fingertip_link"/>
+      <xacro:if value="${jaw_xacro_prop == 'standard'}" >
+        <origin xyz="-0.028 0.0 0.047" rpy="0 0 0"/>
+      </xacro:if>
+    </joint>
+    <!--
+    <xacro:robotiq_hande_transmission prefix="${prefix}"/>
+    <xacro:if value="$(arg use_fake_hardware)">
+      <xacro:robotiq_hande_ros2_control name="robotiq_hande_ros2_control" prefix="${prefix}" use_fake_hardware="$(arg use_fake_hardware)"/>
+    </xacro:if>
+    -->
   </xacro:macro>
 </robot>

Commit message: Adding if statements for different grippers.

File: urdf/robotiq_hande.urdf.xacro (robot description, xacro)
@@ -49,15 +49,20 @@
       </inertial>
       <visual>
-        <origin rpy="0 0 0" xyz="0 0 0"/>
-        <geometry>
-          <mesh filename="package://robotiq_hande_description/meshes/finger_2.dae" scale="0.001 0.001 0.001"/>
-        </geometry>
-        <material name="${prefix}dark_gray"/>
+        <xacro:if value="${jaw_xacro_prop == 'standard'}" >
+          <origin xyz="0.0 0.0 0.0" rpy="0 0 0"/>
+          <geometry>
+            <mesh filename="package://robotiq_hande_description/meshes/finger_2.dae" scale="0.001 0.001 0.001"/>
+          </geometry>
+          <material name="${prefix}dark_gray"/>
+        </xacro:if>
       </visual>
       <collision>
-        <origin rpy="0 0 0" xyz="0 0 0"/>
-        <geometry>
-          <mesh filename="package://robotiq_hande_description/meshes/finger_2.dae" scale="0.001 0.001 0.001"/>
-        </geometry>
+        <xacro:if value="${jaw_xacro_prop == 'standard'}" >
+          <origin xyz="0.0 0.0 0.0" rpy="0 0 0"/>
+          <geometry>
+            <mesh filename="package://robotiq_hande_description/meshes/finger_2.dae" scale="0.001 0.001 0.001"/>
+          </geometry>
+          <material name="${prefix}dark_gray"/>
+        </xacro:if>
       </collision>
     </link>
@@ -69,15 +74,20 @@
       </inertial>
       <visual>
-        <origin rpy="0 0 0" xyz="0 0 0"/>
-        <geometry>
-          <mesh filename="package://robotiq_hande_description/meshes/finger_1.dae" scale="0.001 0.001 0.001"/>
-        </geometry>
-        <material name="${prefix}dark_gray"/>
+        <xacro:if value="${jaw_xacro_prop == 'standard'}" >
+          <origin xyz="0.0 0.0 0.0" rpy="0 0 0"/>
+          <geometry>
+            <mesh filename="package://robotiq_hande_description/meshes/finger_1.dae" scale="0.001 0.001 0.001"/>
+          </geometry>
+          <material name="${prefix}dark_gray"/>
+        </xacro:if>
       </visual>
       <collision>
-        <origin rpy="0 0 0" xyz="0 0 0"/>
-        <geometry>
-          <mesh filename="package://robotiq_hande_description/meshes/finger_1.dae" scale="0.001 0.001 0.001"/>
-        </geometry>
+        <xacro:if value="${jaw_xacro_prop == 'standard'}" >
+          <origin xyz="0.0 0.0 0.0" rpy="0 0 0"/>
+          <geometry>
+            <mesh filename="package://robotiq_hande_description/meshes/finger_1.dae" scale="0.001 0.001 0.001"/>
+          </geometry>
+          <material name="${prefix}dark_gray"/>
+        </xacro:if>
       </collision>
     </link>

Commit message: Debugging fixes.

File: urdf/robotiq_hande.urdf.xacro (robot description, xacro)
@@ -40,4 +40,5 @@
           <mesh filename="package://robotiq_hande_description/meshes/hand-e.dae" scale="0.001 0.001 0.001"/>
         </geometry>
+        <material name="${prefix}black"/>
       </collision>
     </link>
@@ -52,5 +53,5 @@
           <origin xyz="0.0 0.0 0.0" rpy="0 0 0"/>
           <geometry>
-            <mesh filename="package://robotiq_hande_description/meshes/finger_2.dae" scale="0.001 0.001 0.001"/>
+            <mesh filename="package://robotiq_hande_description/meshes/finger_2.stl" scale="0.001 0.001 0.001"/>
           </geometry>
           <material name="${prefix}dark_gray"/>
@@ -61,5 +62,5 @@
           <origin xyz="0.0 0.0 0.0" rpy="0 0 0"/>
           <geometry>
-            <mesh filename="package://robotiq_hande_description/meshes/finger_2.dae" scale="0.001 0.001 0.001"/>
+            <mesh filename="package://robotiq_hande_description/meshes/finger_2.stl" scale="0.001 0.001 0.001"/>
           </geometry>
           <material name="${prefix}dark_gray"/>
@@ -77,5 +78,5 @@
           <origin xyz="0.0 0.0 0.0" rpy="0 0 0"/>
           <geometry>
-            <mesh filename="package://robotiq_hande_description/meshes/finger_1.dae" scale="0.001 0.001 0.001"/>
+            <mesh filename="package://robotiq_hande_description/meshes/finger_1.stl" scale="0.001 0.001 0.001"/>
           </geometry>
           <material name="${prefix}dark_gray"/>
@@ -86,5 +87,5 @@
           <origin xyz="0.0 0.0 0.0" rpy="0 0 0"/>
           <geometry>
-            <mesh filename="package://robotiq_hande_description/meshes/finger_1.dae" scale="0.001 0.001 0.001"/>
+            <mesh filename="package://robotiq_hande_description/meshes/finger_1.stl" scale="0.001 0.001 0.001"/>
           </geometry>
           <material name="${prefix}dark_gray"/>
