Commit message: Updating for ROS2 Humble control.

File: urdf/robotiq_hande_ros2_control.xacro (robot description, xacro)
@@ -1,21 +1,40 @@
 <?xml version="1.0"?>
 <robot xmlns:xacro="http://www.ros.org/wiki/xacro">
- <xacro:macro name="robotiq_hande_ros2_control" params="name prefix use_fake_hardware:=false">
-  <ros2_control name="${name}" type="system">
-    <hardware>
-      <xacro:if value="${use_fake_hardware}">
-        <plugin>fake_components/GenericSystem</plugin>
-      </xacro:if>
-    </hardware>
-    <joint name="${prefix}finger_1_joint">
-      <param name="initial_position">0.00</param>
-      <command_interface name="position">
-        <param name="min">0.00</param>
-        <param name="max">0.05</param>
-      </command_interface>
-      <state_interface name="position"/>
-      <state_interface name="velocity"/>
-    </joint>
-  </ros2_control>
- </xacro:macro>
+  <xacro:macro name="robotiq_hande_ros2_control" params="
+      name:=robotiq
+      prefix
+      use_fake_hardware:=false
+      fake_sensor_commands:=false
+      com_port:=/dev/ttyUSB0">
+    <ros2_control name="${name}" type="system">
+      <hardware>
+        <xacro:if value="${use_fake_hardware}">
+          <plugin>fake_components/GenericSystem</plugin>
+        </xacro:if>
+        <xacro:unless value="${use_fake_hardware}">
+            <plugin>robotiq_driver/RobotiqGripperHardwareInterface</plugin>
+            <param name="gripper_closed_position">0.7929</param>
+            <param name="COM_port">${com_port}</param>
+            <param name="gripper_speed_multiplier">1.0</param>
+            <param name="gripper_force_multiplier">0.5</param>
+        </xacro:unless>
+      </hardware>
+      <joint name="${prefix}finger_1_joint">
+        <param name="initial_position">0.00</param>
+        <command_interface name="position">
+          <param name="min">0.00</param>
+          <param name="max">0.05</param>
+        </command_interface>
+        <state_interface name="position"/>
+        <state_interface name="velocity"/>
+      </joint>
+      <!-- Only add this with fake hardware mode -->
+      <xacro:command_interface value="${use_fake_hardware}">
+          <gpio name="reactivate_gripper">
+              <command_interface name="reactivate_gripper_cmd" />
+              <command_interface name="reactivate_gripper_response" />
+          </gpio>
+      </xacroif>
+    </ros2_control>
+  </xacro:macro>
 </robot>
