Commit message: Changes to work with the ROS2 control driver.

File: urdf/robotiq_hande.ros2_control.xacro (robot description, xacro)
@@ -14,5 +14,5 @@
         <xacro:unless value="${use_fake_hardware}">
             <plugin>robotiq_driver/RobotiqGripperHardwareInterface</plugin>
-            <param name="gripper_closed_position">0.7929</param>
+            <param name="gripper_closed_position">0.059</param>
             <param name="COM_port">${com_port}</param>
             <param name="gripper_speed_multiplier">1.0</param>

File: urdf/robotiq_hande.xacro (robot description, xacro)
@@ -1,12 +1,176 @@
 <?xml version="1.0"?>
-<robot xmlns:xacro="http://wiki.ros.org/xacro" name="robotiq_hande">
-  <xacro:arg name="name" default="robotiq_hande"/>
-  <xacro:arg name="prefix" default="" />
+<robot xmlns:xacro="http://ros.org/wiki/xacro">
   <xacro:arg name="jaw_xacro" default="standard" />
   <xacro:arg name="use_fake_hardware" default="false" />
-  <xacro:include filename="$(find robotiq_hande_description)/urdf/robotiq_hande.urdf.xacro"/>
-  <link name="world"/>
-  <xacro:robotiq_hande name="$(arg name)" prefix="$(arg prefix)" parent="world" use_fake_hardware="$(arg use_fake_hardware)" com_port="/dev/ttyUSB1">
-    <origin xyz="0 0 0" rpy="0 0 0"/>
-  </xacro:robotiq_hande>
+  <xacro:property name="jaw_xacro_prop" value="$(arg jaw_xacro)" />
+  <xacro:include filename="$(find robotiq_hande_description)/urdf/robotiq_hande_transmission.xacro"/>
+  <xacro:include filename="$(find robotiq_hande_description)/urdf/robotiq_hande.ros2_control.xacro"/>
+  <xacro:macro name="robotiq_hande" params="
+    name:=robotiq_hande
+    prefix
+    parent
+    *origin
+    use_fake_hardware:=false
+    fake_sensor_commands:=false
+    com_port:=/dev/ttyUSB1">
+    <material name="${prefix}dark_gray">
+      <color rgba="0.2 0.2 0.2 1"/>
+    </material>
+    <material name="${prefix}black">
+      <color rgba="0 0 0 1"/>
+    </material>
+    <!-- ros2 control instance -->
+    <xacro:robotiq_hande_ros2_control
+        name="${name}"
+        prefix="${prefix}"
+        use_fake_hardware="${use_fake_hardware}"
+        fake_sensor_commands="${fake_sensor_commands}"
+        com_port="${com_port}"
+        />
+    <joint name="${prefix}gripper_base_joint" type="fixed">
+      <parent link="${parent}"/>
+      <child link="${prefix}gripper_base_link"/>
+      <xacro:insert_block name="origin"/>
+    </joint>
+    <link name="${prefix}gripper_base_link">
+      <inertial>
+        <origin xyz="0 0 0.04607" rpy="0 0 0" />
+        <mass value="0.86387" />
+        <inertia ixx="1017560E-9" ixy="0" ixz="2235E-9" iyy="1028041E-9" iyz="0" izz="489810E-9" />
+      </inertial>
+      <visual>
+        <origin xyz="0 0 0" rpy="0 0 0" />
+        <geometry>
+          <mesh filename="package://robotiq_hande_description/meshes/hand-e.dae" scale="0.001 0.001 0.001"/>
+        </geometry>
+        <material name="${prefix}black"/>
+      </visual>
+      <collision>
+        <origin xyz="0 0 0" rpy="0 0 0" />
+        <geometry>
+          <mesh filename="package://robotiq_hande_description/meshes/hand-e.dae" scale="0.001 0.001 0.001"/>
+        </geometry>
+        <material name="${prefix}black"/>
+      </collision>
+    </link>
+    <link name="${prefix}finger_1_link">
+      <inertial>
+        <origin rpy="0 0 0" xyz="-0.02262 0.00759 0.00738"/>
+        <mass value="0.03804"/>
+        <inertia ixx="13567E-9" ixy="1849E-9" ixz="-3622E-9" iyy="15784E-9" iyz="-3616E-9" izz="7478E-9"/>
+      </inertial>
+      <visual>
+        <xacro:if value="${jaw_xacro_prop == 'standard'}" >
+          <origin xyz="0.0 0.0 0.0" rpy="0 0 0"/>
+          <geometry>
+            <mesh filename="package://robotiq_hande_description/meshes/finger_2.stl" scale="0.001 0.001 0.001"/>
+          </geometry>
+          <material name="${prefix}dark_gray"/>
+        </xacro:if>
+      </visual>
+      <collision>
+        <xacro:if value="${jaw_xacro_prop == 'standard'}" >
+          <origin xyz="0.0 0.0 0.0" rpy="0 0 0"/>
+          <geometry>
+            <mesh filename="package://robotiq_hande_description/meshes/finger_2.stl" scale="0.001 0.001 0.001"/>
+          </geometry>
+          <material name="${prefix}dark_gray"/>
+        </xacro:if>
+      </collision>
+    </link>
+    <link name="${prefix}finger_2_link">
+      <inertial>
+        <origin rpy="0 0 0" xyz="0.02262 -0.00759 0.00738"/>
+        <mass value="0.03804"/>
+        <inertia ixx="13567E-9" ixy="1849E-9" ixz="3622E-9" iyy="15784E-9" iyz="3616E-9" izz="7478E-9"/>
+      </inertial>
+      <visual>
+        <xacro:if value="${jaw_xacro_prop == 'standard'}" >
+          <origin xyz="0.0 0.0 0.0" rpy="0 0 0"/>
+          <geometry>
+            <mesh filename="package://robotiq_hande_description/meshes/finger_1.stl" scale="0.001 0.001 0.001"/>
+          </geometry>
+          <material name="${prefix}dark_gray"/>
+        </xacro:if>
+      </visual>
+      <collision>
+        <xacro:if value="${jaw_xacro_prop == 'standard'}" >
+          <origin xyz="0.0 0.0 0.0" rpy="0 0 0"/>
+          <geometry>
+            <mesh filename="package://robotiq_hande_description/meshes/finger_1.stl" scale="0.001 0.001 0.001"/>
+          </geometry>
+          <material name="${prefix}dark_gray"/>
+        </xacro:if>
+      </collision>
+    </link>
+    <joint name="${prefix}finger_1_joint" type="prismatic">
+      <origin rpy="0 0 0" xyz="0 0 0.099"/>
+      <parent link="${prefix}gripper_base_link"/>
+      <child link="${prefix}finger_1_link"/>
+      <axis xyz="1 0 0"/>
+      <limit effort="130" lower="0" upper="0.025" velocity="0.15"/>
+    </joint>
+    <joint name="${prefix}finger_2_joint" type="prismatic">
+      <origin rpy="0 0 0" xyz="0 0 0.099"/>
+      <parent link="${prefix}gripper_base_link"/>
+      <child link="${prefix}finger_2_link"/>
+      <axis xyz="-1 0 0"/>
+      <limit effort="130" lower="0" upper="0.025" velocity="0.15"/>
+      <mimic joint="${prefix}finger_1_joint" multiplier="1" offset="0"/>
+    </joint>
+    <link name="${prefix}grasp_frame">
+      <visual>
+        <geometry>
+          <sphere radius="0.007"/>
+        </geometry>
+        <material name="${prefix}_green">
+          <color rgba="0 1.0 0 1.0"/>
+        </material>
+      </visual>
+    </link>
+    <joint name="${prefix}grasp_frame_joint" type="fixed">
+      <parent link="${prefix}gripper_base_link"/>
+      <child link="${prefix}grasp_frame"/>
+      <xacro:if value="${jaw_xacro_prop == 'standard'}" >
+        <origin xyz="0.0 0.0 0.135" rpy="0 0 0"/>
+      </xacro:if>
+    </joint>
+    <link name="${prefix}push_frame">
+      <visual>
+        <geometry>
+          <box size="0.014 0.014 0.014"/>
+        </geometry>
+        <material name="${prefix}_red">
+          <color rgba="1.0 0 0 1.0"/>
+        </material>
+      </visual>
+    </link>
+    <joint name="${prefix}push_frame_joint" type="fixed">
+      <parent link="${prefix}gripper_base_link"/>
+      <child link="${prefix}push_frame"/>
+      <xacro:if value="${jaw_xacro_prop == 'standard'}" >
+        <origin xyz="0.0 0.0 0.147" rpy="0 0 0"/>
+      </xacro:if>
+    </joint>
+    <!--Calibration frame-->
+    <link name="${prefix}gripper_calibration_link"/>
+    <joint name="${prefix}gripper_finger_base_joint" type="fixed">
+      <parent link="${prefix}gripper_base_link"/>
+      <child link="${prefix}gripper_calibration_link"/>
+      <origin xyz="0.0 0.0 0.099" rpy="0 0 0"/>
+    </joint>
+    <!--Fingertip frames-->
+    <link name="${prefix}finger_1_fingertip_link"/>
+    <joint name="${prefix}finger_1_fingertip_joint" type="fixed">
+      <parent link="${prefix}finger_1_link"/>
+      <child link="${prefix}finger_1_fingertip_link"/>
+      <xacro:if value="${jaw_xacro_prop == 'standard'}" >
+        <origin xyz="-0.028 0.0 0.047" rpy="0 0 0"/>
+      </xacro:if>
+    </joint>
+    <xacro:robotiq_hande_transmission prefix="${prefix}"/>
+    <xacro:if value="$(arg use_fake_hardware)">
+      <xacro:robotiq_hande_ros2_control name="robotiq_hande_ros2_control" prefix="${prefix}" use_fake_hardware="$(arg use_fake_hardware)"/>
+    </xacro:if>
+  </xacro:macro>
 </robot>
