Commit message: Switching some joint locations around for ros2_control.

File: urdf/robotiq_hande.xacro (robot description, xacro)
@@ -13,5 +13,6 @@
     use_fake_hardware:=false
     fake_sensor_commands:=false
-    com_port:=/dev/ttyUSB1">
+    com_port:=/dev/ttyUSB1
+    max_finger_distance:=0.059">
     <material name="${prefix}dark_gray">
       <color rgba="0.2 0.2 0.2 1"/>
@@ -105,15 +106,15 @@
     </link>
     <joint name="${prefix}finger_1_joint" type="prismatic">
-      <origin rpy="0 0 0" xyz="0 0 0.099"/>
+      <origin rpy="0 0 0" xyz="${max_finger_distance / 2} 0 0.099"/>
       <parent link="${prefix}gripper_base_link"/>
       <child link="${prefix}finger_1_link"/>
-      <axis xyz="1 0 0"/>
+      <axis xyz="-1 0 0"/>
       <limit effort="130" lower="0" upper="0.025" velocity="0.15"/>
     </joint>
     <joint name="${prefix}finger_2_joint" type="prismatic">
-      <origin rpy="0 0 0" xyz="0 0 0.099"/>
+      <origin rpy="0 0 0" xyz="${-max_finger_distance / 2}  0 0.099"/>
       <parent link="${prefix}gripper_base_link"/>
       <child link="${prefix}finger_2_link"/>
-      <axis xyz="-1 0 0"/>
+      <axis xyz="1 0 0"/>
       <limit effort="130" lower="0" upper="0.025" velocity="0.15"/>
       <mimic joint="${prefix}finger_1_joint" multiplier="1" offset="0"/>

Commit message: Adding new fingers and adjusting xacro.

File: urdf/robotiq_hande.xacro (robot description, xacro)
@@ -65,5 +65,5 @@
           <origin xyz="0.0 0.0 0.0" rpy="0 0 0"/>
           <geometry>
-            <mesh filename="package://robotiq_hande_description/meshes/finger_2.stl" scale="0.001 0.001 0.001"/>
+            <mesh filename="package://robotiq_hande_description/meshes/hande_fngr_nail_v2.stl" />
           </geometry>
           <material name="${prefix}dark_gray"/>
@@ -74,5 +74,5 @@
           <origin xyz="0.0 0.0 0.0" rpy="0 0 0"/>
           <geometry>
-            <mesh filename="package://robotiq_hande_description/meshes/finger_2.stl" scale="0.001 0.001 0.001"/>
+            <mesh filename="package://robotiq_hande_description/meshes/hande_fngr_nail_v2.stl"/>
           </geometry>
           <material name="${prefix}dark_gray"/>
@@ -90,5 +90,5 @@
           <origin xyz="0.0 0.0 0.0" rpy="0 0 0"/>
           <geometry>
-            <mesh filename="package://robotiq_hande_description/meshes/finger_1.stl" scale="0.001 0.001 0.001"/>
+            <mesh filename="package://robotiq_hande_description/meshes/hande_fngr_nail_v2.stl"/>
           </geometry>
           <material name="${prefix}dark_gray"/>
@@ -99,5 +99,5 @@
           <origin xyz="0.0 0.0 0.0" rpy="0 0 0"/>
           <geometry>
-            <mesh filename="package://robotiq_hande_description/meshes/finger_1.stl" scale="0.001 0.001 0.001"/>
+            <mesh filename="package://robotiq_hande_description/meshes/hande_fngr_nail_v2.stl"/>
           </geometry>
           <material name="${prefix}dark_gray"/>
@@ -106,12 +106,12 @@
     </link>
     <joint name="${prefix}finger_1_joint" type="prismatic">
-      <origin rpy="0 0 0" xyz="${max_finger_distance / 2} 0 0.099"/>
+      <origin rpy="${pi/2} 0 0" xyz="0 -0.003 0.099"/>
       <parent link="${prefix}gripper_base_link"/>
       <child link="${prefix}finger_1_link"/>
-      <axis xyz="-1 0 0"/>
+      <axis xyz="1 0 0"/>
       <limit effort="130" lower="0" upper="0.025" velocity="0.15"/>
     </joint>
     <joint name="${prefix}finger_2_joint" type="prismatic">
-      <origin rpy="0 0 0" xyz="${-max_finger_distance / 2}  0 0.099"/>
+      <origin rpy="${pi/2} 0 ${pi}" xyz="0 0.003 0.099"/>
       <parent link="${prefix}gripper_base_link"/>
       <child link="${prefix}finger_2_link"/>

Commit message: Minor adjustment.

File: urdf/robotiq_hande.xacro (robot description, xacro)
@@ -106,5 +106,5 @@
     </link>
     <joint name="${prefix}finger_1_joint" type="prismatic">
-      <origin rpy="${pi/2} 0 0" xyz="0 -0.003 0.099"/>
+      <origin rpy="${pi/2} 0 0" xyz="0 -0.0032 0.099"/>
       <parent link="${prefix}gripper_base_link"/>
       <child link="${prefix}finger_1_link"/>
@@ -113,5 +113,5 @@
     </joint>
     <joint name="${prefix}finger_2_joint" type="prismatic">
-      <origin rpy="${pi/2} 0 ${pi}" xyz="0 0.003 0.099"/>
+      <origin rpy="${pi/2} 0 ${pi}" xyz="0 0.0032 0.099"/>
       <parent link="${prefix}gripper_base_link"/>
       <child link="${prefix}finger_2_link"/>

Commit message: Updating push and grasp frames.

File: urdf/robotiq_hande.xacro (robot description, xacro)
@@ -134,5 +134,5 @@
       <child link="${prefix}grasp_frame"/>
       <xacro:if value="${jaw_xacro_prop == 'standard'}" >
-        <origin xyz="0.0 0.0 0.135" rpy="0 0 0"/>
+        <origin xyz="0.0 0.0 0.148" rpy="0 0 0"/>
       </xacro:if>
     </joint>
@@ -151,5 +151,5 @@
       <child link="${prefix}push_frame"/>
       <xacro:if value="${jaw_xacro_prop == 'standard'}" >
-        <origin xyz="0.0 0.0 0.147" rpy="0 0 0"/>
+        <origin xyz="0.0 0.0 0.16" rpy="0 0 0"/>
       </xacro:if>
     </joint>

Commit message: Changing the push markers.

File: urdf/robotiq_hande.xacro (robot description, xacro)
@@ -4,4 +4,7 @@
   <xacro:arg name="use_fake_hardware" default="false" />
   <xacro:property name="jaw_xacro_prop" value="$(arg jaw_xacro)" />
+  <xacro:property name="finger_length" default="0.060" />
+  <xacro:property name="push_marker_length" default="0.015" />
+  <xacro:property name="marker_opacity" default="0.25" />
   <xacro:include filename="$(find robotiq_hande_description)/urdf/robotiq_hande_transmission.xacro"/>
   <xacro:include filename="$(find robotiq_hande_description)/urdf/robotiq_hande.ros2_control.xacro"/>
@@ -126,5 +129,5 @@
         </geometry>
         <material name="${prefix}_green">
-          <color rgba="0 1.0 0 1.0"/>
+          <color rgba="0 1.0 0 ${marker_opacity}"/>
         </material>
       </visual>
@@ -137,19 +140,36 @@
       </xacro:if>
     </joint>
-    <link name="${prefix}push_frame">
+    <link name="${prefix}push_frame_1">
       <visual>
         <geometry>
-          <box size="0.014 0.014 0.014"/>
+          <box size="${push_marker_length / 4} ${push_marker_length} ${push_marker_length / 4}"/>
         </geometry>
         <material name="${prefix}_red">
-          <color rgba="1.0 0 0 1.0"/>
+          <color rgba="1.0 0 0 ${marker_opacity}"/>
         </material>
       </visual>
     </link>
-    <joint name="${prefix}push_frame_joint" type="fixed">
-      <parent link="${prefix}gripper_base_link"/>
-      <child link="${prefix}push_frame"/>
+    <joint name="${prefix}push_frame_1_joint" type="fixed">
+      <parent link="${prefix}finger_1_link"/>
+      <child link="${prefix}push_frame_1"/>
       <xacro:if value="${jaw_xacro_prop == 'standard'}" >
-        <origin xyz="0.0 0.0 0.16" rpy="0 0 0"/>
+        <origin xyz="0.002 ${finger_length + push_marker_length / 2} -${push_marker_length / 4}" rpy="0 0 0"/>
+      </xacro:if>
+    </joint>
+    <link name="${prefix}push_frame_2">
+      <visual>
+        <geometry>
+          <box size="${push_marker_length / 4} ${push_marker_length} ${push_marker_length / 4}"/>
+        </geometry>
+        <material name="${prefix}_red">
+          <color rgba="1.0 0 0 ${marker_opacity}"/>
+        </material>
+      </visual>
+    </link>
+    <joint name="${prefix}push_frame_2_joint" type="fixed">
+      <parent link="${prefix}finger_2_link"/>
+      <child link="${prefix}push_frame_2"/>
+      <xacro:if value="${jaw_xacro_prop == 'standard'}" >
+        <origin xyz="0.002 ${finger_length + push_marker_length / 2} -${push_marker_length / 4}" rpy="0 0 0"/>
       </xacro:if>
     </joint>

Commit message: Altering the push frame markers a little bit.

File: urdf/robotiq_hande.xacro (robot description, xacro)
@@ -4,6 +4,6 @@
   <xacro:arg name="use_fake_hardware" default="false" />
   <xacro:property name="jaw_xacro_prop" value="$(arg jaw_xacro)" />
-  <xacro:property name="finger_length" default="0.060" />
-  <xacro:property name="push_marker_length" default="0.015" />
+  <xacro:property name="finger_length" default="0.0605" />
+  <xacro:property name="push_marker_size" default="0.01" />
   <xacro:property name="marker_opacity" default="0.25" />
   <xacro:include filename="$(find robotiq_hande_description)/urdf/robotiq_hande_transmission.xacro"/>
@@ -142,6 +142,7 @@
     <link name="${prefix}push_frame_1">
       <visual>
+        <origin xyz="0.0 ${push_marker_size / 8} 0.0" rpy="0 0 0"/>
         <geometry>
-          <box size="${push_marker_length / 4} ${push_marker_length} ${push_marker_length / 4}"/>
+          <box size="${push_marker_size} ${push_marker_size / 4} ${push_marker_size}"/>
         </geometry>
         <material name="${prefix}_red">
@@ -154,11 +155,12 @@
       <child link="${prefix}push_frame_1"/>
       <xacro:if value="${jaw_xacro_prop == 'standard'}" >
-        <origin xyz="0.002 ${finger_length + push_marker_length / 2} -${push_marker_length / 4}" rpy="0 0 0"/>
+        <origin xyz="0.002 ${finger_length} -0.003" rpy="0 0 0"/>
       </xacro:if>
     </joint>
     <link name="${prefix}push_frame_2">
       <visual>
+        <origin xyz="0.0 ${push_marker_size / 8} 0.0" rpy="0 0 0"/>
         <geometry>
-          <box size="${push_marker_length / 4} ${push_marker_length} ${push_marker_length / 4}"/>
+          <box size="${push_marker_size} ${push_marker_size / 4} ${push_marker_size}"/>
         </geometry>
         <material name="${prefix}_red">
@@ -171,5 +173,5 @@
       <child link="${prefix}push_frame_2"/>
       <xacro:if value="${jaw_xacro_prop == 'standard'}" >
-        <origin xyz="0.002 ${finger_length + push_marker_length / 2} -${push_marker_length / 4}" rpy="0 0 0"/>
+        <origin xyz="0.002 ${finger_length} -0.003" rpy="0 0 0"/>
       </xacro:if>
     </joint>
