Commit message: Altering the push frame markers slightly.

File: dextivr_hande_description/urdf/fngr_v2_m_grasp_push_frames.xacro (robot description, xacro)
@@ -7,5 +7,5 @@
     grasp_distance:=${(170.350-8)/1000.0}
     finger_length:=0.0730250
-    push_marker_size:=0.01">
+    push_marker_size:=0.005">
     <link name="${tf_prefix}grasp_frame">
       <visual>
@@ -25,7 +25,7 @@
     <link name="${tf_prefix}push_frame_1">
       <visual>
-        <origin xyz="0.0 0.0 0.0" rpy="0 0 0"/>
+        <origin xyz="0.0 0.0 ${push_marker_size / 4}" rpy="0 0 0"/>
         <geometry>
-          <box size="${push_marker_size} ${push_marker_size} ${push_marker_size / 4}"/>
+          <box size="${push_marker_size} ${push_marker_size} ${push_marker_size / 2}"/>
         </geometry>
         <material name="${tf_prefix}_red">
@@ -41,7 +41,7 @@
     <link name="${tf_prefix}push_frame_2">
       <visual>
-        <origin xyz="0.0 0.0 0.0" rpy="0 0 0"/>
+        <origin xyz="0.0 0.0 ${push_marker_size / 4}" rpy="0 0 0"/>
         <geometry>
-          <box size="${push_marker_size} ${push_marker_size} ${push_marker_size / 4}"/>
+          <box size="${push_marker_size} ${push_marker_size} ${push_marker_size / 2}"/>
         </geometry>
         <material name="${tf_prefix}_red">

Commit message: Adding center_push frame.

File: dextivr_hande_description/urdf/fngr_v2_m_grasp_push_frames.xacro (robot description, xacro)
@@ -55,4 +55,21 @@
       <origin xyz="0.0041 0.00325 ${finger_length}" rpy="0 0 ${pi}"/>
     </joint>
+    <link name="${tf_prefix}center_push_frame">
+      <visual>
+        <origin xyz="0.0 0.0 ${push_marker_size / 4}" rpy="0 0 0"/>
+        <geometry>
+          <box size="${push_marker_size} ${push_marker_size} ${push_marker_size / 2}"/>
+        </geometry>
+        <material name="${tf_prefix}_red">
+          <color rgba="1.0 0 0 ${marker_opacity}"/>
+        </material>
+      </visual>
+    </link>
+    <!-- The 0.01 is for the finger mount offset -->
+    <joint name="${tf_prefix}center_push_frame_joint" type="fixed">
+      <parent link="${tf_prefix}gripper_palm_link"/>
+      <child link="${tf_prefix}center_push_frame"/>
+      <origin xyz="0.0 0.0 ${finger_length + 0.0017}" rpy="0 0 0"/>
+    </joint>
   </xacro:macro>
 </robot>
