Commit message: Viewing works again.

File: dextivr_hande_description/urdf/dextivr_hande.urdf.xacro (robot description, xacro)
@@ -6,10 +6,10 @@
   <xacro:arg name="com_port" default="/dev/ttyACM0" />
   <xacro:arg name="marker_opacity" default="0.25" />
-  <xacro:arg name="grasp_distance" default="0.130" />
-  <xacro:arg name="finger_length" default="0.046" />
+  <xacro:arg name="grasp_distance" default="0.148" />
+  <xacro:arg name="finger_length" default="0.0605" />
   <xacro:arg name="push_marker_size" default="0.01" />
   <xacro:include filename="$(find robotiq_hande_description)/urdf/robotiq_hande.xacro"/>
   <xacro:include filename="$(find dextivr_hande_description)/urdf/hande_fingers_fngr_nail_v2.xacro"/>
-  <xacro:include filename="$(find robotiq_hande_description)/urdf/grasp_push_frames.xacro"/>
+  <xacro:include filename="$(find dextivr_hande_description)/urdf/fngr_nail_v2_grasp_push_frames.xacro"/>
   <link name="world"/>
   <xacro:robotiq_hande name="$(arg name)" prefix="$(arg prefix)" parent="world" use_fake_hardware="$(arg use_fake_hardware)" com_port="$(arg com_port)">

File: dextivr_hande_description/urdf/hande_fingers_fngr_nail_v2.xacro (robot description, xacro)
@@ -3,5 +3,12 @@
   <xacro:macro name="hande_fingers" params="
     name:=''
-    prefix:=''">
+    prefix:=''
+    mount_x:=0.0
+    mount_y:=0.0032
+    mount_z:=0.099
+    mount_roll:=${pi/2}
+    mount_pitch:=0.0
+    mount_yaw:=${pi}
+    scale:=0.001">
     <link name="${prefix}finger_1_link">
       <visual>
@@ -37,5 +44,5 @@
     </link>
     <joint name="${prefix}finger_1_joint" type="prismatic">
-      <origin rpy="${mount_roll} ${mount_pitch} ${mount_yaw}" xyz="${-mount_x} ${-mount_y} ${mount_z}"/>
+      <origin rpy="${mount_roll} ${mount_pitch} ${mount_yaw}" xyz="${mount_x} ${mount_y} ${mount_z}"/>
       <parent link="${prefix}gripper_base_link"/>
       <child link="${prefix}finger_1_link"/>
@@ -44,5 +51,5 @@
     </joint>
     <joint name="${prefix}finger_2_joint" type="prismatic">
-      <origin rpy="${mount_roll} ${mount_pitch} ${mount_yaw + pi}" xyz="${mount_x} ${mount_y} ${mount_z}"/>
+      <origin rpy="${mount_roll} ${mount_pitch} ${mount_yaw + pi}" xyz="${mount_x} ${-mount_y} ${mount_z}"/>
       <parent link="${prefix}gripper_base_link"/>
       <child link="${prefix}finger_2_link"/>

Commit message: Ease of use changes for MR.

File: dextivr_hande_description/urdf/dextivr_hande.urdf.xacro (robot description, xacro)
@@ -5,16 +5,16 @@
   <xacro:arg name="use_fake_hardware" default="false" />
   <xacro:arg name="com_port" default="/dev/ttyACM0" />
-  <xacro:arg name="marker_opacity" default="0.25" />
-  <xacro:arg name="grasp_distance" default="0.148" />
-  <xacro:arg name="finger_length" default="0.0605" />
-  <xacro:arg name="push_marker_size" default="0.01" />
+  <xacro:arg name="finger_xacro" default="fngr_nail_v2" />
+  <xacro:property name="finger_type_prop" value="$(arg finger_xacro)" />
   <xacro:include filename="$(find robotiq_hande_description)/urdf/robotiq_hande.xacro"/>
-  <xacro:include filename="$(find dextivr_hande_description)/urdf/hande_fingers_fngr_nail_v2.xacro"/>
-  <xacro:include filename="$(find dextivr_hande_description)/urdf/fngr_nail_v2_grasp_push_frames.xacro"/>
   <link name="world"/>
   <xacro:robotiq_hande name="$(arg name)" prefix="$(arg prefix)" parent="world" use_fake_hardware="$(arg use_fake_hardware)" com_port="$(arg com_port)">
     <origin xyz="0 0 0" rpy="0 0 0"/>
   </xacro:robotiq_hande>
+  <xacro:if value="${finger_type_prop == 'fngr_nail_v2'}">
+    <xacro:include filename="$(find dextivr_hande_description)/urdf/hande_fingers_fngr_nail_v2.xacro"/>
+    <xacro:include filename="$(find dextivr_hande_description)/urdf/fngr_nail_v2_grasp_push_frames.xacro"/>
+  </xacro:if>
   <xacro:hande_fingers name="$(arg name)" prefix="$(arg prefix)"/>
-  <xacro:grasp_push_frames name="$(arg name)" prefix="$(arg prefix)" marker_opacity="$(arg marker_opacity)" grasp_distance="$(arg grasp_distance)" finger_length="$(arg finger_length)" push_marker_size="$(arg push_marker_size)"/>
+  <xacro:grasp_push_frames name="$(arg name)" prefix="$(arg prefix)"/>
 </robot>

Commit message: Updates for push frames.

File: dextivr_hande_description/urdf/dextivr_hande.urdf.xacro (robot description, xacro)
@@ -2,12 +2,12 @@
 <robot xmlns:xacro="http://wiki.ros.org/xacro" name="robotiq_hande">
   <xacro:arg name="name" default="RobotiqGripperHandeHardwareInterface"/>
-  <xacro:arg name="prefix" default="" />
+  <xacro:arg name="tf_prefix" default="" />
   <xacro:arg name="use_fake_hardware" default="false" />
   <xacro:arg name="com_port" default="/dev/ttyACM0" />
-  <xacro:arg name="finger_xacro" default="fngr_nail_v2_m" />
+  <xacro:arg name="finger_xacro" default="fngr_v2_m" />
   <xacro:property name="finger_type_prop" value="$(arg finger_xacro)" />
   <xacro:include filename="$(find robotiq_hande_description)/urdf/robotiq_hande.xacro"/>
   <link name="world"/>
-  <xacro:robotiq_hande name="$(arg name)" prefix="$(arg prefix)" parent="world" use_fake_hardware="$(arg use_fake_hardware)" com_port="$(arg com_port)">
+  <xacro:robotiq_hande name="$(arg name)" tf_prefix="$(arg tf_prefix)" parent="world" use_fake_hardware="$(arg use_fake_hardware)" com_port="$(arg com_port)">
     <origin xyz="0 0 0" rpy="0 0 0"/>
   </xacro:robotiq_hande>
@@ -17,10 +17,10 @@
     <xacro:include filename="$(find dextivr_hande_description)/urdf/fngr_nail_v2_grasp_push_frames.xacro"/>
   </xacro:if>
-  <xacro:if value="${finger_type_prop == 'fngr_nail_v2_m'}">
+  <xacro:if value="${finger_type_prop == 'fngr_v2_m'}">
     <xacro:include filename="$(find dextivr_hande_description)/urdf/hande_fingers_v2_m.xacro"/>
     <xacro:include filename="$(find dextivr_hande_description)/urdf/fngr_v2_m_grasp_push_frames.xacro"/>
   </xacro:if>
   <!--Run the xacros from the files included above-->
-  <xacro:hande_fingers name="$(arg name)" prefix="$(arg prefix)"/>
-  <xacro:grasp_push_frames name="$(arg name)" prefix="$(arg prefix)"/>
+  <xacro:hande_fingers name="$(arg name)" tf_prefix="$(arg tf_prefix)"/>
+  <xacro:grasp_push_frames name="$(arg name)" tf_prefix="$(arg tf_prefix)"/>
 </robot>

File: dextivr_hande_description/urdf/fngr_nail_v2_grasp_push_frames.xacro (robot description, xacro)
@@ -3,55 +3,55 @@
   <xacro:macro name="grasp_push_frames" params="
     name:=''
-    prefix:=''
+    tf_prefix:=''
     marker_opacity:=0.25
     grasp_distance:=0.148
     finger_length:=0.0605
     push_marker_size:=0.01">
-    <link name="${prefix}grasp_frame">
+    <link name="${tf_prefix}grasp_frame">
       <visual>
         <geometry>
           <sphere radius="0.007"/>
         </geometry>
-        <material name="${prefix}_green">
+        <material name="${tf_prefix}_green">
           <color rgba="0 1.0 0 ${marker_opacity}"/>
         </material>
       </visual>
     </link>
-    <joint name="${prefix}grasp_frame_joint" type="fixed">
-      <parent link="${prefix}gripper_base_link"/>
-      <child link="${prefix}grasp_frame"/>
+    <joint name="${tf_prefix}grasp_frame_joint" type="fixed">
+      <parent link="${tf_prefix}gripper_base_link"/>
+      <child link="${tf_prefix}grasp_frame"/>
       <origin xyz="0.0 0.0 ${grasp_distance}" rpy="0 0 0"/>
     </joint>
-    <link name="${prefix}push_frame_1">
+    <link name="${tf_prefix}push_frame_1">
       <visual>
-        <origin xyz="0.0 ${push_marker_size / 8} 0.0" rpy="0 0 0"/>
+        <origin xyz="0.0 0.0 ${push_marker_size / 8}" rpy="0 0 0"/>
         <geometry>
-          <box size="${push_marker_size} ${push_marker_size / 4} ${push_marker_size}"/>
+          <box size="${push_marker_size} ${push_marker_size} ${push_marker_size / 4}"/>
         </geometry>
-        <material name="${prefix}_red">
+        <material name="${tf_prefix}_red">
           <color rgba="1.0 0 0 ${marker_opacity}"/>
         </material>
       </visual>
     </link>
-    <joint name="${prefix}push_frame_1_joint" type="fixed">
-      <parent link="${prefix}finger_1_link"/>
-      <child link="${prefix}push_frame_1"/>
-      <origin xyz="0.0 ${finger_length} -0.003" rpy="0 0 0"/>
+    <joint name="${tf_prefix}push_frame_1_joint" type="fixed">
+      <parent link="${tf_prefix}finger_1_link"/>
+      <child link="${tf_prefix}push_frame_1"/>
+      <origin xyz="0.0 ${finger_length} -0.003" rpy="${-pi/2} ${pi} 0"/>
     </joint>
-    <link name="${prefix}push_frame_2">
+    <link name="${tf_prefix}push_frame_2">
       <visual>
-        <origin xyz="0.0 ${push_marker_size / 8} 0.0" rpy="0 0 0"/>
+        <origin xyz="0.0 0.0 ${push_marker_size / 8}" rpy="0 0 0"/>
         <geometry>
-          <box size="${push_marker_size} ${push_marker_size / 4} ${push_marker_size}"/>
+          <box size="${push_marker_size} ${push_marker_size} ${push_marker_size / 4}"/>
         </geometry>
-        <material name="${prefix}_red">
+        <material name="${tf_prefix}_red">
           <color rgba="1.0 0 0 ${marker_opacity}"/>
         </material>
       </visual>
     </link>
-    <joint name="${prefix}push_frame_2_joint" type="fixed">
-      <parent link="${prefix}finger_2_link"/>
-      <child link="${prefix}push_frame_2"/>
-      <origin xyz="0.0 ${finger_length} -0.003" rpy="0 0 0"/>
+    <joint name="${tf_prefix}push_frame_2_joint" type="fixed">
+      <parent link="${tf_prefix}finger_2_link"/>
+      <child link="${tf_prefix}push_frame_2"/>
+      <origin xyz="0.0 ${finger_length} -0.003" rpy="${-pi/2} 0 0"/>
     </joint>
   </xacro:macro>

File: dextivr_hande_description/urdf/fngr_v2_m_grasp_push_frames.xacro (robot description, xacro)
@@ -3,25 +3,25 @@
   <xacro:macro name="grasp_push_frames" params="
     name:=''
-    prefix:=''
+    tf_prefix:=''
     marker_opacity:=0.25
     grasp_distance:=${(170.350-8)/1000.0}
     finger_length:=0.0730250
     push_marker_size:=0.01">
-    <link name="${prefix}grasp_frame">
+    <link name="${tf_prefix}grasp_frame">
       <visual>
         <geometry>
           <sphere radius="0.007"/>
         </geometry>
-        <material name="${prefix}_green">
+        <material name="${tf_prefix}_green">
           <color rgba="0 1.0 0 ${marker_opacity}"/>
         </material>
       </visual>
     </link>
-    <joint name="${prefix}grasp_frame_joint" type="fixed">
-      <parent link="${prefix}gripper_base_link"/>
-      <child link="${prefix}grasp_frame"/>
+    <joint name="${tf_prefix}grasp_frame_joint" type="fixed">
+      <parent link="${tf_prefix}gripper_base_link"/>
+      <child link="${tf_prefix}grasp_frame"/>
       <origin xyz="0.0 0.0 ${grasp_distance}" rpy="0 0 0"/>
     </joint>
-    <link name="${prefix}push_frame_1">
+    <link name="${tf_prefix}push_frame_1">
       <visual>
         <origin xyz="0.0 0.0 0.0" rpy="0 0 0"/>
@@ -29,15 +29,15 @@
           <box size="${push_marker_size} ${push_marker_size} ${push_marker_size / 4}"/>
         </geometry>
-        <material name="${prefix}_red">
+        <material name="${tf_prefix}_red">
           <color rgba="1.0 0 0 ${marker_opacity}"/>
         </material>
       </visual>
     </link>
-    <joint name="${prefix}push_frame_1_joint" type="fixed">
-      <parent link="${prefix}finger_1_link"/>
-      <child link="${prefix}push_frame_1"/>
+    <joint name="${tf_prefix}push_frame_1_joint" type="fixed">
+      <parent link="${tf_prefix}finger_1_link"/>
+      <child link="${tf_prefix}push_frame_1"/>
       <origin xyz="0.0041 0.00325 ${finger_length}" rpy="0 0 0"/>
     </joint>
-    <link name="${prefix}push_frame_2">
+    <link name="${tf_prefix}push_frame_2">
       <visual>
         <origin xyz="0.0 0.0 0.0" rpy="0 0 0"/>
@@ -45,13 +45,13 @@
           <box size="${push_marker_size} ${push_marker_size} ${push_marker_size / 4}"/>
         </geometry>
-        <material name="${prefix}_red">
+        <material name="${tf_prefix}_red">
           <color rgba="1.0 0 0 ${marker_opacity}"/>
         </material>
       </visual>
     </link>
-    <joint name="${prefix}push_frame_2_joint" type="fixed">
-      <parent link="${prefix}finger_2_link"/>
-      <child link="${prefix}push_frame_2"/>
-      <origin xyz="0.0041 0.00325 ${finger_length}" rpy="0 0 0"/>
+    <joint name="${tf_prefix}push_frame_2_joint" type="fixed">
+      <parent link="${tf_prefix}finger_2_link"/>
+      <child link="${tf_prefix}push_frame_2"/>
+      <origin xyz="0.0041 0.00325 ${finger_length}" rpy="0 0 ${pi}"/>
     </joint>
   </xacro:macro>

File: dextivr_hande_description/urdf/hande_fingers_fngr_nail_v2.xacro (robot description, xacro)
@@ -3,5 +3,5 @@
   <xacro:macro name="hande_fingers" params="
     name:=''
-    prefix:=''
+    tf_prefix:=''
     mount_x:=0.0
     mount_y:=0.0032
@@ -11,50 +11,62 @@
     mount_yaw:=${pi}
     scale:=0.001">
-    <link name="${prefix}finger_1_link">
+    <link name="${tf_prefix}finger_1_link">
+      <!--TODO set proper inertia-->
+      <inertial>
+        <origin rpy="0 0 0" xyz="0.0 0.0 0.0"/>
+        <mass value="0.0"/>
+        <inertia ixx="0.0" ixy="0.0" ixz="0.0" iyy="0.0" iyz="0.0" izz="0.0"/>
+      </inertial>
       <visual>
           <origin xyz="0.0 0.0 0.0" rpy="0 0 0"/>
           <geometry>
-            <mesh filename="package://dextivr_hande_description/meshes/hande_fngr_nail_v2.stl" />
+            <mesh filename="package://dextivr_hande_description/meshes/visual/hande_fngr_nail_v2.stl" />
           </geometry>
-          <material name="${prefix}dark_gray"/>
+          <material name="${tf_prefix}dark_gray"/>
       </visual>
       <collision>
           <origin xyz="0.0 0.0 0.0" rpy="0 0 0"/>
           <geometry>
-            <mesh filename="package://dextivr_hande_description/meshes/hande_fngr_nail_v2.stl"/>
+            <mesh filename="package://dextivr_hande_description/meshes/collision/hande_fngr_nail_v2.stl"/>
           </geometry>
-          <material name="${prefix}dark_gray"/>
+          <material name="${tf_prefix}dark_gray"/>
       </collision>
     </link>
-    <link name="${prefix}finger_2_link">
+    <link name="${tf_prefix}finger_2_link">
+      <!--TODO set proper inertia-->
+      <inertial>
+        <origin rpy="0 0 0" xyz="0.0 0.0 0.0"/>
+        <mass value="0.0"/>
+        <inertia ixx="0.0" ixy="0.0" ixz="0.0" iyy="0.0" iyz="0.0" izz="0.0"/>
+      </inertial>
       <visual>
           <origin xyz="0.0 0.0 0.0" rpy="0 0 0"/>
           <geometry>
-            <mesh filename="package://dextivr_hande_description/meshes/hande_fngr_nail_v2.stl"/>
+            <mesh filename="package://dextivr_hande_description/meshes/visual/hande_fngr_nail_v2.stl"/>
           </geometry>
-          <material name="${prefix}dark_gray"/>
+          <material name="${tf_prefix}dark_gray"/>
       </visual>
       <collision>
           <origin xyz="0.0 0.0 0.0" rpy="0 0 0"/>
           <geometry>
-            <mesh filename="package://dextivr_hande_description/meshes/hande_fngr_nail_v2.stl"/>
+            <mesh filename="package://dextivr_hande_description/meshes/collision/hande_fngr_nail_v2.stl"/>
           </geometry>
-          <material name="${prefix}dark_gray"/>
+          <material name="${tf_prefix}dark_gray"/>
       </collision>
     </link>
-    <joint name="${prefix}finger_1_joint" type="prismatic">
+    <joint name="${tf_prefix}finger_1_joint" type="prismatic">
       <origin rpy="${mount_roll} ${mount_pitch} ${mount_yaw}" xyz="${mount_x} ${mount_y} ${mount_z}"/>
-      <parent link="${prefix}gripper_base_link"/>
-      <child link="${prefix}finger_1_link"/>
+      <parent link="${tf_prefix}gripper_base_link"/>
+      <child link="${tf_prefix}finger_1_link"/>
       <axis xyz="1 0 0"/>
       <limit effort="130" lower="0" upper="0.025" velocity="0.15"/>
     </joint>
-    <joint name="${prefix}finger_2_joint" type="prismatic">
+    <joint name="${tf_prefix}finger_2_joint" type="prismatic">
       <origin rpy="${mount_roll} ${mount_pitch} ${mount_yaw + pi}" xyz="${mount_x} ${-mount_y} ${mount_z}"/>
-      <parent link="${prefix}gripper_base_link"/>
-      <child link="${prefix}finger_2_link"/>
+      <parent link="${tf_prefix}gripper_base_link"/>
+      <child link="${tf_prefix}finger_2_link"/>
       <axis xyz="1 0 0"/>
       <limit effort="130" lower="0" upper="0.025" velocity="0.15"/>
-      <mimic joint="${prefix}finger_1_joint" multiplier="1" offset="0"/>
+      <mimic joint="${tf_prefix}finger_1_joint" multiplier="1" offset="0"/>
     </joint>
   </xacro:macro>

File: dextivr_hande_description/urdf/hande_fingers_v2_m.xacro (robot description, xacro)
@@ -1,7 +1,8 @@
 <?xml version="1.0"?>
 <robot xmlns:xacro="http://ros.org/wiki/xacro">
+  <!--Scaled from mm to m-->
   <xacro:macro name="hande_fingers" params="
     name:=''
-    prefix:=''
+    tf_prefix:=''
     mount_x:=${2.01401 * 0.001}
     mount_y:=${-3.25000 * 0.001}
@@ -11,50 +12,62 @@
     mount_yaw:=${radians(0)}
     scale:=0.001">
-    <link name="${prefix}finger_1_link">
+    <link name="${tf_prefix}finger_1_link">
+      <!--TODO set proper inertia-->
+      <inertial>
+        <origin rpy="0 0 0" xyz="0.0 0.0 0.0"/>
+        <mass value="0.0"/>
+        <inertia ixx="0.0" ixy="0.0" ixz="0.0" iyy="0.0" iyz="0.0" izz="0.0"/>
+      </inertial>
       <visual>
           <origin xyz="0.0 0.0 0.0" rpy="0 0 0"/>
           <geometry>
-            <mesh filename="package://dextivr_hande_description/meshes/imetro_finger_v2_m_vis.dae" />
+            <mesh filename="package://dextivr_hande_description/meshes/visual/imetro_finger_v2_m_vis.dae" />
           </geometry>
-          <material name="${prefix}dark_gray"/>
+          <material name="${tf_prefix}dark_gray"/>
       </visual>
       <collision>
           <origin xyz="0.0 0.0 0.0" rpy="0 0 0"/>
           <geometry>
-            <mesh filename="package://dextivr_hande_description/meshes/imetro_finger_v2_m_col.dae"/>
+            <mesh filename="package://dextivr_hande_description/meshes/collision/imetro_finger_v2_m_col.dae"/>
           </geometry>
-          <material name="${prefix}dark_gray"/>
+          <material name="${tf_prefix}dark_gray"/>
       </collision>
     </link>
-    <link name="${prefix}finger_2_link">
+    <link name="${tf_prefix}finger_2_link">
+      <!--TODO set proper inertia-->
+      <inertial>
+        <origin rpy="0 0 0" xyz="0.0 0.0 0.0"/>
+        <mass value="0.0"/>
+        <inertia ixx="0.0" ixy="0.0" ixz="0.0" iyy="0.0" iyz="0.0" izz="0.0"/>
+      </inertial>
       <visual>
           <origin xyz="0.0 0.0 0.0" rpy="0 0 0"/>
           <geometry>
-            <mesh filename="package://dextivr_hande_description/meshes/imetro_finger_v2_m_vis.dae" />
+            <mesh filename="package://dextivr_hande_description/meshes/visual/imetro_finger_v2_m_vis.dae" />
           </geometry>
-          <material name="${prefix}dark_gray"/>
+          <material name="${tf_prefix}dark_gray"/>
       </visual>
       <collision>
           <origin xyz="0.0 0.0 0.0" rpy="0 0 0"/>
           <geometry>
-            <mesh filename="package://dextivr_hande_description/meshes/imetro_finger_v2_m_col.dae"/>
+            <mesh filename="package://dextivr_hande_description/meshes/collision/imetro_finger_v2_m_col.dae"/>
           </geometry>
-          <material name="${prefix}dark_gray"/>
+          <material name="${tf_prefix}dark_gray"/>
       </collision>
     </link>
-    <joint name="${prefix}finger_1_joint" type="prismatic">
+    <joint name="${tf_prefix}finger_1_joint" type="prismatic">
       <origin rpy="${mount_roll} ${mount_pitch} ${mount_yaw}" xyz="${mount_x} ${mount_y} ${mount_z}"/>
-      <parent link="${prefix}gripper_base_link"/>
-      <child link="${prefix}finger_1_link"/>
+      <parent link="${tf_prefix}gripper_base_link"/>
+      <child link="${tf_prefix}finger_1_link"/>
       <axis xyz="1 0 0"/>
       <limit effort="130" lower="0" upper="0.025" velocity="0.15"/>
     </joint>
-    <joint name="${prefix}finger_2_joint" type="prismatic">
+    <joint name="${tf_prefix}finger_2_joint" type="prismatic">
       <origin rpy="${mount_roll} ${mount_pitch} ${mount_yaw + pi}" xyz="${-mount_x} ${-mount_y} ${mount_z}"/>
-      <parent link="${prefix}gripper_base_link"/>
-      <child link="${prefix}finger_2_link"/>
+      <parent link="${tf_prefix}gripper_base_link"/>
+      <child link="${tf_prefix}finger_2_link"/>
       <axis xyz="1 0 0"/>
       <limit effort="130" lower="0" upper="0.025" velocity="0.15"/>
-      <mimic joint="${prefix}finger_1_joint" multiplier="1" offset="0"/>
+      <mimic joint="${tf_prefix}finger_1_joint" multiplier="1" offset="0"/>
     </joint>
   </xacro:macro>

Commit message: Cleaning some things for adding the stylus to CLR.

File: dextivr_hande_description/urdf/dextivr_hande.urdf.xacro (robot description, xacro)
@@ -6,21 +6,15 @@
   <xacro:arg name="com_port" default="/dev/ttyACM0" />
   <xacro:arg name="finger_xacro" default="fngr_v2_m" />
+  <material name="$(arg tf_prefix)dark_gray">
+    <color rgba="0.2 0.2 0.2 1"/>
+  </material>
+  <material name="$(arg tf_prefix)black">
+    <color rgba="0 0 0 1"/>
+  </material>
   <xacro:property name="finger_type_prop" value="$(arg finger_xacro)" />
-  <xacro:include filename="$(find robotiq_hande_description)/urdf/robotiq_hande.xacro"/>
+  <xacro:include filename="$(find dextivr_hande_description)/urdf/dextivr_hande.xacro"/>
   <link name="world"/>
-  <xacro:robotiq_hande name="$(arg name)" tf_prefix="$(arg tf_prefix)" parent="world" use_fake_hardware="$(arg use_fake_hardware)" com_port="$(arg com_port)">
+  <xacro:dextivr_hande name="$(arg name)" tf_prefix="$(arg tf_prefix)" parent="world" use_fake_hardware="$(arg use_fake_hardware)" com_port="$(arg com_port)">
     <origin xyz="0 0 0" rpy="0 0 0"/>
-  </xacro:robotiq_hande>
-  <!--If statements for the various types of gripper fingers-->
-  <xacro:if value="${finger_type_prop == 'fngr_nail_v2'}">
-    <xacro:include filename="$(find dextivr_hande_description)/urdf/hande_fingers_fngr_nail_v2.xacro"/>
-    <xacro:include filename="$(find dextivr_hande_description)/urdf/fngr_nail_v2_grasp_push_frames.xacro"/>
-  </xacro:if>
-  <xacro:if value="${finger_type_prop == 'fngr_v2_m'}">
-    <xacro:include filename="$(find dextivr_hande_description)/urdf/hande_fingers_v2_m.xacro"/>
-    <xacro:include filename="$(find dextivr_hande_description)/urdf/fngr_v2_m_grasp_push_frames.xacro"/>
-  </xacro:if>
-  <!--Run the xacros from the files included above-->
-  <xacro:hande_fingers name="$(arg name)" tf_prefix="$(arg tf_prefix)"/>
-  <xacro:grasp_push_frames name="$(arg name)" tf_prefix="$(arg tf_prefix)"/>
+  </xacro:dextivr_hande>
 </robot>
