Commit message: Cleanup.

File: dextivr_hande_description/urdf/dextivr_hande.urdf.xacro (robot description, xacro)
@@ -6,4 +6,5 @@
   <xacro:arg name="com_port" default="/dev/ttyACM0" />
   <xacro:arg name="finger_xacro" default="fngr_v2_m" />
+  <xacro:arg name="marker_opacity" default="0.5" />
   <material name="$(arg tf_prefix)dark_gray">
     <color rgba="0.2 0.2 0.2 1"/>
@@ -11,4 +12,10 @@
   <material name="$(arg tf_prefix)black">
     <color rgba="0 0 0 1"/>
+  </material>
+  <material name="$(arg tf_prefix)red_marker">
+    <color rgba="1 0 0 $(arg marker_opacity)"/>
+  </material>
+  <material name="$(arg tf_prefix)green_marker">
+    <color rgba="0 1 0 $(arg marker_opacity)"/>
   </material>
   <xacro:property name="finger_type_prop" value="$(arg finger_xacro)" />

File: dextivr_hande_description/urdf/dextivr_hande.xacro (robot description, xacro)
@@ -8,5 +8,6 @@
     use_fake_hardware:=false
     fake_sensor_commands:=false
-    com_port:=/dev/ttyUSB0">
+    com_port:=/dev/ttyUSB0
+    marker_opacity:=0.5">
   <xacro:property name="finger_type_prop" value="$(arg finger_xacro)" />
   <xacro:include filename="$(find robotiq_hande_description)/urdf/robotiq_hande.xacro"/>

File: dextivr_hande_description/urdf/fngr_nail_v2_grasp_push_frames.xacro (robot description, xacro)
@@ -13,7 +13,5 @@
           <sphere radius="0.007"/>
         </geometry>
-        <material name="${tf_prefix}_green">
-          <color rgba="0 1.0 0 ${marker_opacity}"/>
-        </material>
+        <material name="${tf_prefix}green_marker"/>
       </visual>
     </link>
@@ -29,7 +27,5 @@
           <box size="${push_marker_size} ${push_marker_size} ${push_marker_size / 4}"/>
         </geometry>
-        <material name="${tf_prefix}_red">
-          <color rgba="1.0 0 0 ${marker_opacity}"/>
-        </material>
+        <material name="${tf_prefix}red_marker"/>
       </visual>
     </link>
@@ -45,7 +41,5 @@
           <box size="${push_marker_size} ${push_marker_size} ${push_marker_size / 4}"/>
         </geometry>
-        <material name="${tf_prefix}_red">
-          <color rgba="1.0 0 0 ${marker_opacity}"/>
-        </material>
+        <material name="${tf_prefix}red_marker"/>
       </visual>
     </link>
@@ -61,7 +55,5 @@
           <box size="${push_marker_size} ${push_marker_size} ${push_marker_size / 4}"/>
         </geometry>
-        <material name="${tf_prefix}_red">
-          <color rgba="1.0 0 0 ${marker_opacity}"/>
-        </material>
+        <material name="${tf_prefix}red_marker"/>
       </visual>
     </link>

File: dextivr_hande_description/urdf/fngr_v2_m_grasp_push_frames.xacro (robot description, xacro)
@@ -13,7 +13,5 @@
           <sphere radius="0.007"/>
         </geometry>
-        <material name="${tf_prefix}_green">
-          <color rgba="0 1.0 0 ${marker_opacity}"/>
-        </material>
+        <material name="${tf_prefix}green_marker"/>
       </visual>
     </link>
@@ -29,7 +27,5 @@
           <box size="${push_marker_size} ${push_marker_size} ${push_marker_size / 2}"/>
         </geometry>
-        <material name="${tf_prefix}_red">
-          <color rgba="1.0 0 0 ${marker_opacity}"/>
-        </material>
+        <material name="${tf_prefix}red_marker"/>
       </visual>
     </link>
@@ -45,7 +41,5 @@
           <box size="${push_marker_size} ${push_marker_size} ${push_marker_size / 2}"/>
         </geometry>
-        <material name="${tf_prefix}_red">
-          <color rgba="1.0 0 0 ${marker_opacity}"/>
-        </material>
+        <material name="${tf_prefix}red_marker"/>
       </visual>
     </link>
@@ -61,7 +55,5 @@
           <box size="${push_marker_size} ${push_marker_size} ${push_marker_size / 2}"/>
         </geometry>
-        <material name="${tf_prefix}_red">
-          <color rgba="1.0 0 0 ${marker_opacity}"/>
-        </material>
+        <material name="${tf_prefix}red_marker"/>
       </visual>
     </link>

Commit message: Cleaning up for chonkur stylus.

File: dextivr_hande_description/urdf/dextivr_hande.urdf.xacro (robot description, xacro)
@@ -22,5 +22,5 @@
   <xacro:include filename="$(find dextivr_hande_description)/urdf/dextivr_hande.xacro"/>
   <link name="world"/>
-  <xacro:dextivr_hande name="$(arg name)" tf_prefix="$(arg tf_prefix)" parent="world" use_fake_hardware="$(arg use_fake_hardware)" com_port="$(arg com_port)">
+  <xacro:dextivr_hande name="$(arg name)" tf_prefix="$(arg tf_prefix)" parent="world" use_fake_hardware="$(arg use_fake_hardware)" com_port="$(arg com_port)" finger_xacro="$(arg finger_xacro)">
     <origin xyz="0 0 0" rpy="0 0 0"/>
   </xacro:dextivr_hande>

File: dextivr_hande_description/urdf/dextivr_hande.xacro (robot description, xacro)
@@ -2,5 +2,5 @@
 <robot xmlns:xacro="http://wiki.ros.org/xacro">
   <xacro:macro name="dextivr_hande" params="
-    name
+    name:=RobotiqGripperHandeHardwareInterface
     tf_prefix
     parent
@@ -9,22 +9,22 @@
     fake_sensor_commands:=false
     com_port:=/dev/ttyUSB0
-    marker_opacity:=0.5">
-  <xacro:property name="finger_type_prop" value="$(arg finger_xacro)" />
+    marker_opacity:=0.5
+    finger_xacro:=fngr_v2_m">
   <xacro:include filename="$(find robotiq_hande_description)/urdf/robotiq_hande.xacro"/>
-  <xacro:robotiq_hande name="$(arg name)" tf_prefix="$(arg tf_prefix)" parent="${parent}" use_fake_hardware="$(arg use_fake_hardware)" com_port="$(arg com_port)">
+  <xacro:robotiq_hande name="${name}" tf_prefix="${tf_prefix}" parent="${parent}" use_fake_hardware="${use_fake_hardware}" com_port="${com_port}">
     <origin xyz="0 0 0" rpy="0 0 0"/>
   </xacro:robotiq_hande>
   <!--If statements for the various types of gripper fingers-->
-  <xacro:if value="${finger_type_prop == 'fngr_nail_v2'}">
+  <xacro:if value="${finger_xacro == 'fngr_nail_v2'}">
     <xacro:include filename="$(find dextivr_hande_description)/urdf/hande_fingers_fngr_nail_v2.xacro"/>
     <xacro:include filename="$(find dextivr_hande_description)/urdf/fngr_nail_v2_grasp_push_frames.xacro"/>
   </xacro:if>
-  <xacro:if value="${finger_type_prop == 'fngr_v2_m'}">
+  <xacro:if value="${finger_xacro == 'fngr_v2_m'}">
     <xacro:include filename="$(find dextivr_hande_description)/urdf/hande_fingers_v2_m.xacro"/>
     <xacro:include filename="$(find dextivr_hande_description)/urdf/fngr_v2_m_grasp_push_frames.xacro"/>
   </xacro:if>
   <!--Run the xacros from the files included above-->
-  <xacro:hande_fingers name="$(arg name)" tf_prefix="$(arg tf_prefix)"/>
-  <xacro:grasp_push_frames name="$(arg name)" tf_prefix="$(arg tf_prefix)"/>
+  <xacro:hande_fingers name="${name}" tf_prefix="${tf_prefix}"/>
+  <xacro:grasp_push_frames name="${name}" tf_prefix="${tf_prefix}"/>
   </xacro:macro>
 </robot>

Commit message: propagating marker_opacity arg

File: dextivr_hande_description/urdf/dextivr_hande.urdf.xacro (robot description, xacro)
@@ -22,5 +22,5 @@
   <xacro:include filename="$(find dextivr_hande_description)/urdf/dextivr_hande.xacro"/>
   <link name="world"/>
-  <xacro:dextivr_hande name="$(arg name)" tf_prefix="$(arg tf_prefix)" parent="world" use_fake_hardware="$(arg use_fake_hardware)" com_port="$(arg com_port)" finger_xacro="$(arg finger_xacro)">
+  <xacro:dextivr_hande name="$(arg name)" tf_prefix="$(arg tf_prefix)" parent="world" use_fake_hardware="$(arg use_fake_hardware)" com_port="$(arg com_port)" finger_xacro="$(arg finger_xacro)" marker_opacity="$(arg marker_opacity)">
     <origin xyz="0 0 0" rpy="0 0 0"/>
   </xacro:dextivr_hande>

File: dextivr_hande_description/urdf/dextivr_hande.xacro (robot description, xacro)
@@ -29,6 +29,6 @@
   </xacro:if>
   <!--Run the xacros from the files included above-->
-  <xacro:hande_fingers name="${name}" tf_prefix="${tf_prefix}"/>
-  <xacro:grasp_push_frames name="${name}" tf_prefix="${tf_prefix}"/>
+  <xacro:hande_fingers name="${name}" tf_prefix="${tf_prefix}" />
+  <xacro:grasp_push_frames name="${name}" tf_prefix="${tf_prefix}" marker_opacity="${marker_opacity}"/>
   </xacro:macro>
 </robot>

File: dextivr_hande_description/urdf/fngr_v2_m_grasp_push_frames.xacro (robot description, xacro)
@@ -13,5 +13,7 @@
           <sphere radius="0.007"/>
         </geometry>
-        <material name="${tf_prefix}green_marker"/>
+        <material name="${tf_prefix}green_marker">
+          <color rgba="0 1.0 0 ${marker_opacity}"/>
+        </material>
       </visual>
     </link>
@@ -27,5 +29,7 @@
           <box size="${push_marker_size} ${push_marker_size} ${push_marker_size / 2}"/>
         </geometry>
-        <material name="${tf_prefix}red_marker"/>
+        <material name="${tf_prefix}red_marker">
+          <color rgba="1.0 0 0 ${marker_opacity}"/>
+        </material>
       </visual>
     </link>
@@ -41,5 +45,7 @@
           <box size="${push_marker_size} ${push_marker_size} ${push_marker_size / 2}"/>
         </geometry>
-        <material name="${tf_prefix}red_marker"/>
+        <material name="${tf_prefix}red_marker">
+          <color rgba="1.0 0 0 ${marker_opacity}"/>
+        </material>
       </visual>
     </link>
@@ -55,5 +61,7 @@
           <box size="${push_marker_size} ${push_marker_size} ${push_marker_size / 2}"/>
         </geometry>
-        <material name="${tf_prefix}red_marker"/>
+        <material name="${tf_prefix}red_marker">
+          <color rgba="1.0 0 0 ${marker_opacity}"/>
+        </material>
       </visual>
     </link>

Commit message: fixing non-unique materials error by giving everything its own special little material properties

File: dextivr_hande_description/urdf/dextivr_hande.urdf.xacro (robot description, xacro)
@@ -6,21 +6,16 @@
   <xacro:arg name="com_port" default="/dev/ttyACM0" />
   <xacro:arg name="finger_xacro" default="fngr_v6" />
-  <xacro:arg name="marker_opacity" default="0.5" />
-  <material name="$(arg tf_prefix)dark_gray">
-    <color rgba="0.2 0.2 0.2 1"/>
-  </material>
-  <material name="$(arg tf_prefix)black">
-    <color rgba="0 0 0 1"/>
-  </material>
-  <material name="$(arg tf_prefix)red_marker">
-    <color rgba="1 0 0 $(arg marker_opacity)"/>
-  </material>
-  <material name="$(arg tf_prefix)green_marker">
-    <color rgba="0 1 0 $(arg marker_opacity)"/>
-  </material>
+  <xacro:arg name="marker_opacity" default="0.1" />
   <xacro:property name="finger_type_prop" value="$(arg finger_xacro)" />
   <xacro:include filename="$(find dextivr_hande_description)/urdf/dextivr_hande.xacro"/>
   <link name="world"/>
-  <xacro:dextivr_hande name="$(arg name)" tf_prefix="$(arg tf_prefix)" parent="world" use_fake_hardware="$(arg use_fake_hardware)" com_port="$(arg com_port)" finger_xacro="$(arg finger_xacro)" marker_opacity="$(arg marker_opacity)">
+  <xacro:dextivr_hande
+    name="$(arg name)"
+    tf_prefix="$(arg tf_prefix)"
+    parent="world"
+    use_fake_hardware="$(arg use_fake_hardware)"
+    com_port="$(arg com_port)"
+    finger_xacro="$(arg finger_xacro)"
+    marker_opacity="$(arg marker_opacity)">
     <origin xyz="0 0 0" rpy="0 0 0"/>
   </xacro:dextivr_hande>

File: dextivr_hande_description/urdf/fngr_nail_v2_grasp_push_frames.xacro (robot description, xacro)
@@ -8,4 +8,10 @@
     finger_length:=0.0605
     push_marker_size:=0.01">
+    <material name="$${tf_prefix}fngr_nail_v2_grasp_push_frames_red_marker">
+      <color rgba="1.0 0 0 ${marker_opacity}"/>
+    </material>
+    <material name="${tf_prefix}fngr_nail_v2_grasp_push_frames_green_marker">
+      <color rgba="0 1.0 0 ${marker_opacity}"/>
+    </material>
     <link name="${tf_prefix}grasp_frame">
       <visual>
@@ -13,5 +19,5 @@
           <sphere radius="0.007"/>
         </geometry>
-        <material name="${tf_prefix}green_marker"/>
+        <material name="${tf_prefix}fngr_nail_v2_grasp_push_frames_green_marker"/>
       </visual>
     </link>
@@ -27,5 +33,5 @@
           <box size="${push_marker_size} ${push_marker_size} ${push_marker_size / 4}"/>
         </geometry>
-        <material name="${tf_prefix}red_marker"/>
+        <material name="${tf_prefix}fngr_nail_v2_grasp_push_frames_red_marker"/>
       </visual>
     </link>
@@ -41,5 +47,5 @@
           <box size="${push_marker_size} ${push_marker_size} ${push_marker_size / 4}"/>
         </geometry>
-        <material name="${tf_prefix}red_marker"/>
+        <material name="${tf_prefix}fngr_nail_v2_grasp_push_frames_red_marker"/>
       </visual>
     </link>
@@ -55,5 +61,5 @@
           <box size="${push_marker_size} ${push_marker_size} ${push_marker_size / 4}"/>
         </geometry>
-        <material name="${tf_prefix}red_marker"/>
+        <material name="${tf_prefix}fngr_nail_v2_grasp_push_frames_red_marker"/>
       </visual>
     </link>

File: dextivr_hande_description/urdf/fngr_v2_m_grasp_push_frames.xacro (robot description, xacro)
@@ -8,4 +8,10 @@
     finger_length:=0.0730250
     push_marker_size:=0.005">
+    <material name="${tf_prefix}fngr_v2_m_grasp_push_frames_red_marker">
+      <color rgba="1.0 0 0 ${marker_opacity}"/>
+    </material>
+    <material name="${tf_prefix}fngr_v2_m_grasp_push_frames_green_marker">
+      <color rgba="0 1.0 0 ${marker_opacity}"/>
+    </material>
     <link name="${tf_prefix}grasp_frame">
       <visual>
@@ -13,7 +19,5 @@
           <sphere radius="0.007"/>
         </geometry>
-        <material name="${tf_prefix}green_marker">
-          <color rgba="0 1.0 0 ${marker_opacity}"/>
-        </material>
+        <material name="${tf_prefix}fngr_v2_m_grasp_push_frames_green_marker"/>
       </visual>
     </link>
@@ -29,7 +33,5 @@
           <box size="${push_marker_size} ${push_marker_size} ${push_marker_size / 2}"/>
         </geometry>
-        <material name="${tf_prefix}red_marker">
-          <color rgba="1.0 0 0 ${marker_opacity}"/>
-        </material>
+        <material name="${tf_prefix}fngr_v2_m_grasp_push_frames_red_marker"/>
       </visual>
     </link>
@@ -45,7 +47,5 @@
           <box size="${push_marker_size} ${push_marker_size} ${push_marker_size / 2}"/>
         </geometry>
-        <material name="${tf_prefix}red_marker">
-          <color rgba="1.0 0 0 ${marker_opacity}"/>
-        </material>
+        <material name="${tf_prefix}fngr_v2_m_grasp_push_frames_red_marker"/>
       </visual>
     </link>
@@ -61,7 +61,5 @@
           <box size="${push_marker_size} ${push_marker_size} ${push_marker_size / 2}"/>
         </geometry>
-        <material name="${tf_prefix}red_marker">
-          <color rgba="1.0 0 0 ${marker_opacity}"/>
-        </material>
+        <material name="${tf_prefix}fngr_v2_m_grasp_push_frames_red_marker"/>
       </visual>
     </link>

File: dextivr_hande_description/urdf/hande_fingers_fngr_nail_v2.xacro (robot description, xacro)
@@ -11,4 +11,7 @@
     mount_yaw:=${pi}
     scale:=0.001">
+    <material name="${tf_prefix}hande_fingers_fngr_nail_v2_dark_gray">
+      <color rgba="0.2 0.2 0.2 1"/>
+    </material>
     <link name="${tf_prefix}finger_1_link">
       <!--TODO set proper inertia-->
@@ -23,5 +26,5 @@
             <mesh filename="package://dextivr_hande_description/meshes/visual/hande_fngr_nail_v2.stl" />
           </geometry>
-          <material name="${tf_prefix}dark_gray"/>
+          <material name="${tf_prefix}hande_fingers_fngr_nail_v2_dark_gray"/>
       </visual>
       <collision>
@@ -30,5 +33,5 @@
             <mesh filename="package://dextivr_hande_description/meshes/collision/hande_fngr_nail_v2.stl"/>
           </geometry>
-          <material name="${tf_prefix}dark_gray"/>
+          <material name="${tf_prefix}hande_fingers_fngr_nail_v2_dark_gray"/>
       </collision>
     </link>
@@ -45,5 +48,5 @@
             <mesh filename="package://dextivr_hande_description/meshes/visual/hande_fngr_nail_v2.stl"/>
           </geometry>
-          <material name="${tf_prefix}dark_gray"/>
+          <material name="${tf_prefix}hande_fingers_fngr_nail_v2_dark_gray"/>
       </visual>
       <collision>
@@ -52,5 +55,5 @@
             <mesh filename="package://dextivr_hande_description/meshes/collision/hande_fngr_nail_v2.stl"/>
           </geometry>
-          <material name="${tf_prefix}dark_gray"/>
+          <material name="${tf_prefix}hande_fingers_fngr_nail_v2_dark_gray"/>
       </collision>
     </link>

File: dextivr_hande_description/urdf/hande_fingers_v2_m.xacro (robot description, xacro)
@@ -12,4 +12,7 @@
     mount_yaw:=${radians(0)}
     scale:=0.001">
+    <material name="${tf_prefix}hande_fingers_v2_m_dark_gray">
+      <color rgba="0.2 0.2 0.2 1"/>
+    </material>
     <link name="${tf_prefix}finger_1_link">
       <!--TODO set proper inertia-->
@@ -24,5 +27,5 @@
             <mesh filename="package://dextivr_hande_description/meshes/visual/imetro_finger_v2_m_vis.dae" />
           </geometry>
-          <material name="${tf_prefix}dark_gray"/>
+          <material name="${tf_prefix}hande_fingers_v2_m_dark_gray"/>
       </visual>
       <collision>
@@ -31,5 +34,5 @@
             <mesh filename="package://dextivr_hande_description/meshes/collision/imetro_finger_v2_m_col.dae"/>
           </geometry>
-          <material name="${tf_prefix}dark_gray"/>
+          <material name="${tf_prefix}hande_fingers_v2_m_dark_gray"/>
       </collision>
     </link>
@@ -46,5 +49,5 @@
             <mesh filename="package://dextivr_hande_description/meshes/visual/imetro_finger_v2_m_vis.dae" />
           </geometry>
-          <material name="${tf_prefix}dark_gray"/>
+          <material name="${tf_prefix}hande_fingers_v2_m_dark_gray"/>
       </visual>
       <collision>
@@ -53,5 +56,5 @@
             <mesh filename="package://dextivr_hande_description/meshes/collision/imetro_finger_v2_m_col.dae"/>
           </geometry>
-          <material name="${tf_prefix}dark_gray"/>
+          <material name="${tf_prefix}hande_fingers_v2_m_dark_gray"/>
       </collision>
     </link>

File: dextivr_hande_description/urdf/hande_fingers_v6.xacro (robot description, xacro)
@@ -12,4 +12,7 @@
     mount_yaw:=${radians(0)}
     scale:=0.001">
+    <material name="${tf_prefix}hande_fingers_v6_dark_gray">
+      <color rgba="0.2 0.2 0.2 1"/>
+    </material>
     <link name="${tf_prefix}finger_1_link">
       <!--TODO set proper inertia-->
@@ -24,5 +27,5 @@
             <mesh filename="package://dextivr_hande_description/meshes/visual/finger_v6.stl" />
           </geometry>
-          <material name="${tf_prefix}dark_gray"/>
+          <material name="${tf_prefix}hande_fingers_v6_dark_gray"/>
       </visual>
       <collision>
@@ -31,5 +34,5 @@
             <mesh filename="package://dextivr_hande_description/meshes/collision/finger_v6.stl"/>
           </geometry>
-          <material name="${tf_prefix}dark_gray"/>
+          <material name="${tf_prefix}hande_fingers_v6_dark_gray"/>
       </collision>
     </link>
@@ -46,5 +49,5 @@
             <mesh filename="package://dextivr_hande_description/meshes/visual/finger_v6.stl" />
           </geometry>
-          <material name="${tf_prefix}dark_gray"/>
+          <material name="${tf_prefix}hande_fingers_v6_dark_gray"/>
       </visual>
       <collision>
@@ -53,5 +56,5 @@
             <mesh filename="package://dextivr_hande_description/meshes/collision/finger_v6.stl"/>
           </geometry>
-          <material name="${tf_prefix}dark_gray"/>
+          <material name="${tf_prefix}hande_fingers_v6_dark_gray"/>
       </collision>
     </link>
