Commit message: adjusted the finger width

File: dextivr_hande_description/urdf/hande_fingers_v2_m.xacro (robot description, xacro)
@@ -64,5 +64,5 @@
       <child link="${tf_prefix}finger_1_link"/>
       <axis xyz="1 0 0"/>
-      <limit effort="130" lower="0" upper="0.025" velocity="0.15"/>
+      <limit effort="130" lower="0" upper="0.029" velocity="0.15"/>
     </joint>
     <joint name="${tf_prefix}finger_2_joint" type="prismatic">
@@ -71,5 +71,5 @@
       <child link="${tf_prefix}finger_2_link"/>
       <axis xyz="1 0 0"/>
-      <limit effort="130" lower="0" upper="0.025" velocity="0.15"/>
+      <limit effort="130" lower="0" upper="0.029" velocity="0.15"/>
       <mimic joint="${tf_prefix}finger_1_joint" multiplier="1" offset="0"/>
     </joint>

Commit message: needed to open fingers more

File: dextivr_hande_description/urdf/hande_fingers_v2_m.xacro (robot description, xacro)
@@ -64,5 +64,5 @@
       <child link="${tf_prefix}finger_1_link"/>
       <axis xyz="1 0 0"/>
-      <limit effort="130" lower="0" upper="0.029" velocity="0.15"/>
+      <limit effort="130" lower="0" upper="0.03" velocity="0.15"/>
     </joint>
     <joint name="${tf_prefix}finger_2_joint" type="prismatic">
@@ -71,5 +71,5 @@
       <child link="${tf_prefix}finger_2_link"/>
       <axis xyz="1 0 0"/>
-      <limit effort="130" lower="0" upper="0.029" velocity="0.15"/>
+      <limit effort="130" lower="0" upper="0.03" velocity="0.15"/>
       <mimic joint="${tf_prefix}finger_1_joint" multiplier="1" offset="0"/>
     </joint>

Commit message: Turns out we cant plan to absolute limits

File: dextivr_hande_description/urdf/hande_fingers_v2_m.xacro (robot description, xacro)
@@ -64,5 +64,5 @@
       <child link="${tf_prefix}finger_1_link"/>
       <axis xyz="1 0 0"/>
-      <limit effort="130" lower="0" upper="0.03" velocity="0.15"/>
+      <limit effort="130" lower="0" upper="0.031" velocity="0.15"/>
     </joint>
     <joint name="${tf_prefix}finger_2_joint" type="prismatic">
@@ -71,5 +71,5 @@
       <child link="${tf_prefix}finger_2_link"/>
       <axis xyz="1 0 0"/>
-      <limit effort="130" lower="0" upper="0.03" velocity="0.15"/>
+      <limit effort="130" lower="0" upper="0.031" velocity="0.15"/>
       <mimic joint="${tf_prefix}finger_1_joint" multiplier="1" offset="0"/>
     </joint>
