Commit message: added mass props to fngr v6

File: dextivr_hande_description/urdf/hande_fingers_v6.xacro (robot description, xacro)
@@ -11,14 +11,13 @@
     mount_pitch:=${radians(0)}
     mount_yaw:=${radians(0)}
-    scale:=0.001">
+    scale:=0.001">s
     <material name="${tf_prefix}hande_fingers_v6_dark_gray">
       <color rgba="0.2 0.2 0.2 1"/>
     </material>
     <link name="${tf_prefix}finger_1_link">
-      <!--TODO set proper inertia-->
       <inertial>
         <origin rpy="0 0 0" xyz="0.0 0.0 0.0"/>
-        <mass value="0.0"/>
-        <inertia ixx="0.0" ixy="0.0" ixz="0.0" iyy="0.0" iyz="0.0" izz="0.0"/>
+        <mass value="0.050019846"/>
+        <inertia ixx="0.000060226393" ixy="-0.0000009852757" ixz="-0.00000994007986" iyy="0.000062464751" iyz="-0.0000028146120" izz="0.0000079760530"/>
       </inertial>
       <visual>
@@ -41,6 +40,6 @@
       <inertial>
         <origin rpy="0 0 0" xyz="0.0 0.0 0.0"/>
-        <mass value="0.0"/>
-        <inertia ixx="0.0" ixy="0.0" ixz="0.0" iyy="0.0" iyz="0.0" izz="0.0"/>
+        <mass value="0.050019846"/>
+        <inertia ixx="0.000060226393" ixy="-0.0000009852757" ixz="-0.00000994007986" iyy="0.000062464751" iyz="-0.0000028146120" izz="0.0000079760530"/>
       </inertial>
       <visual>
