Commit message: fix finger inertia (thx tobia)

File: dextivr_hande_description/urdf/hande_fingers_v6.xacro (robot description, xacro)
@@ -17,7 +17,7 @@
     <link name="${tf_prefix}finger_1_link">
       <inertial>
-        <origin rpy="0 0 0" xyz="0.0 0.0 0.0"/>
+        <origin rpy="7.0596949e-03  3.0320393e-05  2.6853115e-02" xyz="0.0 0.0 0.0"/>
         <mass value="0.050019846"/>
-        <inertia ixx="0.000060226393" ixy="-0.0000009852757" ixz="-0.00000994007986" iyy="0.000062464751" iyz="-0.0000028146120" izz="0.0000079760530"/>
+        <inertia ixx="2.3611980e-05" ixy="-9.6469045e-07" ixz="-4.0598189e-07" iyy="2.3361282e-05" iyz="-2.7394321e-06" izz="5.4570651e-06"/>
       </inertial>
       <visual>
@@ -44,7 +44,7 @@
     <link name="${tf_prefix}finger_2_link">
       <inertial>
-        <origin rpy="0 0 0" xyz="0.0 0.0 0.0"/>
+        <origin rpy="7.0596949e-03  3.0320393e-05  2.6853115e-02" xyz="0.0 0.0 0.0"/>
         <mass value="0.050019846"/>
-        <inertia ixx="0.000060226393" ixy="-0.0000009852757" ixz="-0.00000994007986" iyy="0.000062464751" iyz="-0.0000028146120" izz="0.0000079760530"/>
+        <inertia ixx="2.3611980e-05" ixy="-9.6469045e-07" ixz="-4.0598189e-07" iyy="2.3361282e-05" iyz="-2.7394321e-06" izz="5.4570651e-06"/>
       </inertial>
       <visual>
