Commit message: Fixing the origin block.

File: dextivr_hande_description/urdf/dextivr_hande.xacro (robot description, xacro)
@@ -13,5 +13,5 @@
   <xacro:include filename="$(find robotiq_hande_description)/urdf/robotiq_hande.xacro"/>
   <xacro:robotiq_hande name="${name}" tf_prefix="${tf_prefix}" parent="${parent}" use_fake_hardware="${use_fake_hardware}" com_port="${com_port}">
-    <origin xyz="0 0 0" rpy="0 0 0"/>
+    <xacro:insert_block name="origin"/>
   </xacro:robotiq_hande>
   <!--If statements for the various types of gripper fingers-->

Commit message: Add path modifications for mesh files to support gazebo path requirements at launch

File: dextivr_hande_description/urdf/dextivr_hande.xacro (robot description, xacro)
@@ -6,4 +6,5 @@
     parent
     *origin
+    sim_ignition:=false
     use_fake_hardware:=false
     fake_sensor_commands:=false
@@ -11,6 +12,15 @@
     marker_opacity:=0.5
     finger_xacro:=fngr_v6">
+  <!-- if ignition or gazebo - need to use absolute paths instead of relative, applies locally -->
+  <xacro:property name="force_abs_paths" value="$(arg sim_ignition)" />
   <xacro:include filename="$(find robotiq_hande_description)/urdf/robotiq_hande.xacro"/>
-  <xacro:robotiq_hande name="${name}" tf_prefix="${tf_prefix}" parent="${parent}" use_fake_hardware="${use_fake_hardware}" com_port="${com_port}">
+  <xacro:include filename="$(find robotiq_hande_description)/urdf/gen_mesh.xacro"/>
+  <xacro:robotiq_hande
+    name="${name}"
+    tf_prefix="${tf_prefix}"
+    parent="${parent}"
+    sim_ignition="${sim_ignition}"
+    use_fake_hardware="${use_fake_hardware}"
+    com_port="${com_port}">
     <xacro:insert_block name="origin"/>
   </xacro:robotiq_hande>

File: dextivr_hande_description/urdf/hande_fingers_v2_m.xacro (robot description, xacro)
@@ -25,5 +25,8 @@
           <origin xyz="0.0 0.0 0.0" rpy="0 0 0"/>
           <geometry>
-            <mesh filename="package://dextivr_hande_description/meshes/visual/imetro_finger_v2_m_vis.dae" />
+            <xacro:gen_mesh
+              force_abs_path="${force_abs_paths}"
+              pkg_name="dextivr_hande_description"
+              file_path="meshes/visual/imetro_finger_v2_m_vis.dae" />
           </geometry>
           <material name="${tf_prefix}hande_fingers_v2_m_dark_gray"/>

File: dextivr_hande_description/urdf/hande_fingers_v6.xacro (robot description, xacro)
@@ -24,5 +24,8 @@
           <origin xyz="0.0 0.0 0.0" rpy="0 0 0"/>
           <geometry>
-            <mesh filename="package://dextivr_hande_description/meshes/visual/finger_v6.stl" />
+            <xacro:gen_mesh
+              force_abs_path="${force_abs_paths}"
+              pkg_name="dextivr_hande_description"
+              file_path="meshes/visual/finger_v6.stl" />
           </geometry>
           <material name="${tf_prefix}hande_fingers_v6_dark_gray"/>
@@ -31,5 +34,8 @@
           <origin xyz="0.0 0.0 0.0" rpy="0 0 0"/>
           <geometry>
-            <mesh filename="package://dextivr_hande_description/meshes/collision/finger_v6.stl"/>
+            <xacro:gen_mesh
+              force_abs_path="${force_abs_paths}"
+              pkg_name="dextivr_hande_description"
+              file_path="meshes/collision/finger_v6.stl" />
           </geometry>
           <material name="${tf_prefix}hande_fingers_v6_dark_gray"/>
@@ -45,5 +51,8 @@
           <origin xyz="0.0 0.0 0.0" rpy="0 0 0"/>
           <geometry>
-            <mesh filename="package://dextivr_hande_description/meshes/visual/finger_v6.stl" />
+            <xacro:gen_mesh
+              force_abs_path="${force_abs_paths}"
+              pkg_name="dextivr_hande_description"
+              file_path="meshes/visual/finger_v6.stl" />
           </geometry>
           <material name="${tf_prefix}hande_fingers_v6_dark_gray"/>
@@ -52,5 +61,8 @@
           <origin xyz="0.0 0.0 0.0" rpy="0 0 0"/>
           <geometry>
-            <mesh filename="package://dextivr_hande_description/meshes/collision/finger_v6.stl"/>
+            <xacro:gen_mesh
+              force_abs_path="${force_abs_paths}"
+              pkg_name="dextivr_hande_description"
+              file_path="meshes/collision/finger_v6.stl" />
           </geometry>
           <material name="${tf_prefix}hande_fingers_v6_dark_gray"/>

Commit message: updating the sim ignition to reference the macro param, not global arg

File: dextivr_hande_description/urdf/dextivr_hande.xacro (robot description, xacro)
@@ -13,5 +13,5 @@
     finger_xacro:=fngr_v6">
   <!-- if ignition or gazebo - need to use absolute paths instead of relative, applies locally -->
-  <xacro:property name="force_abs_paths" value="$(arg sim_ignition)" />
+  <xacro:property name="force_abs_paths" value="${sim_ignition}" />
   <xacro:include filename="$(find robotiq_hande_description)/urdf/robotiq_hande.xacro"/>
   <xacro:include filename="$(find robotiq_hande_description)/urdf/gen_mesh.xacro"/>
