Commit message: Cleaning up files.

File: dextivr_hande_description/urdf/fngr_nail_v2_grasp_push_frames.xacro (robot description, xacro)
@@ -4,7 +4,7 @@
     name:=''
     prefix:=''
-    marker_opacity:=0.5
-    grasp_distance:=0.130
-    finger_length:=0.046
+    marker_opacity:=0.25
+    grasp_distance:=0.148
+    finger_length:=0.0605
     push_marker_size:=0.01">
     <link name="${prefix}grasp_frame">
@@ -37,5 +37,5 @@
       <parent link="${prefix}finger_1_link"/>
       <child link="${prefix}push_frame_1"/>
-      <origin xyz="0.0 ${finger_length} 0.0" rpy="0 0 0"/>
+      <origin xyz="0.0 ${finger_length} -0.003" rpy="0 0 0"/>
     </joint>
     <link name="${prefix}push_frame_2">
@@ -53,5 +53,5 @@
       <parent link="${prefix}finger_2_link"/>
       <child link="${prefix}push_frame_2"/>
-      <origin xyz="0.0 ${finger_length} 0.0" rpy="0 0 0"/>
+      <origin xyz="0.0 ${finger_length} -0.003" rpy="0 0 0"/>
     </joint>
   </xacro:macro>

Commit message: Adding a central push frame.

File: dextivr_hande_description/urdf/fngr_nail_v2_grasp_push_frames.xacro (robot description, xacro)
@@ -55,4 +55,20 @@
       <origin xyz="0.0 ${finger_length} -0.003" rpy="${-pi/2} 0 0"/>
     </joint>
+    <link name="${tf_prefix}center_push_frame">
+      <visual>
+        <origin xyz="0.0 0.0 ${push_marker_size / 8}" rpy="0 0 0"/>
+        <geometry>
+          <box size="${push_marker_size} ${push_marker_size} ${push_marker_size / 4}"/>
+        </geometry>
+        <material name="${tf_prefix}_red">
+          <color rgba="1.0 0 0 ${marker_opacity}"/>
+        </material>
+      </visual>
+    </link>
+    <joint name="${tf_prefix}center_push_frame_joint" type="fixed">
+      <parent link="${tf_prefix}gripper_palm_link"/>
+      <child link="${tf_prefix}center_push_frame"/>
+      <origin xyz="0.0 0.0 ${finger_length}" rpy="0 0 0"/>
+    </joint>
   </xacro:macro>
 </robot>

Commit message: workaround for hardcoded grasp_link in moveit pro SetADmittanceParams behavior

File: dextivr_hande_description/urdf/fngr_nail_v2_grasp_push_frames.xacro (robot description, xacro)
@@ -25,4 +25,17 @@
       <parent link="${tf_prefix}gripper_base_link"/>
       <child link="${tf_prefix}grasp_frame"/>
+      <origin xyz="0.0 0.0 ${grasp_distance}" rpy="0 0 0"/>
+    </joint>
+    <link name="${tf_prefix}grasp_link">
+      <visual>
+        <geometry>
+          <sphere radius="0.007"/>
+        </geometry>
+        <material name="${tf_prefix}fngr_nail_v2_grasp_push_frames_green_marker"/>
+      </visual>
+    </link>
+    <joint name="${tf_prefix}grasp_link_joint" type="fixed">
+      <parent link="${tf_prefix}gripper_base_link"/>
+      <child link="${tf_prefix}grasp_link"/>
       <origin xyz="0.0 0.0 ${grasp_distance}" rpy="0 0 0"/>
     </joint>

File: dextivr_hande_description/urdf/fngr_v2_m_grasp_push_frames.xacro (robot description, xacro)
@@ -36,4 +36,17 @@
       </visual>
     </link>
+    <link name="${tf_prefix}grasp_link">
+      <visual>
+        <geometry>
+          <sphere radius="0.007"/>
+        </geometry>
+        <material name="${tf_prefix}fngr_nail_v2_grasp_push_frames_green_marker"/>
+      </visual>
+    </link>
+    <joint name="${tf_prefix}grasp_link_joint" type="fixed">
+      <parent link="${tf_prefix}gripper_base_link"/>
+      <child link="${tf_prefix}grasp_link"/>
+      <origin xyz="0.0 0.0 ${grasp_distance}" rpy="0 0 0"/>
+    </joint>
     <joint name="${tf_prefix}push_frame_1_joint" type="fixed">
       <parent link="${tf_prefix}finger_1_link"/>
