Commit message: increase force limit to match datasheet

File: dextivr_hande_description/urdf/hande_fingers_fngr_nail_v2.xacro (robot description, xacro)
@@ -63,5 +63,5 @@
       <child link="${tf_prefix}finger_1_link"/>
       <axis xyz="1 0 0"/>
-      <limit effort="130" lower="0" upper="0.025" velocity="0.15"/>
+      <limit effort="185" lower="0" upper="0.025" velocity="0.15"/>
     </joint>
     <joint name="${tf_prefix}finger_2_joint" type="prismatic">
@@ -70,5 +70,5 @@
       <child link="${tf_prefix}finger_2_link"/>
       <axis xyz="1 0 0"/>
-      <limit effort="130" lower="0" upper="0.025" velocity="0.15"/>
+      <limit effort="185" lower="0" upper="0.025" velocity="0.15"/>
       <mimic joint="${tf_prefix}finger_1_joint" multiplier="1" offset="0"/>
     </joint>

File: dextivr_hande_description/urdf/hande_fingers_v2_m.xacro (robot description, xacro)
@@ -67,5 +67,5 @@
       <child link="${tf_prefix}finger_1_link"/>
       <axis xyz="1 0 0"/>
-      <limit effort="130" lower="0" upper="0.031" velocity="0.15"/>
+      <limit effort="185" lower="0" upper="0.031" velocity="0.15"/>
     </joint>
     <joint name="${tf_prefix}finger_2_joint" type="prismatic">
@@ -74,5 +74,5 @@
       <child link="${tf_prefix}finger_2_link"/>
       <axis xyz="1 0 0"/>
-      <limit effort="130" lower="0" upper="0.031" velocity="0.15"/>
+      <limit effort="185" lower="0" upper="0.031" velocity="0.15"/>
       <mimic joint="${tf_prefix}finger_1_joint" multiplier="1" offset="0"/>
     </joint>

File: dextivr_hande_description/urdf/hande_fingers_v6.xacro (robot description, xacro)
@@ -74,5 +74,5 @@
       <child link="${tf_prefix}finger_1_link"/>
       <axis xyz="1 0 0"/>
-      <limit effort="130" lower="0" upper="0.025" velocity="0.15"/>
+      <limit effort="185" lower="0" upper="0.025" velocity="0.15"/>
     </joint>
     <joint name="${tf_prefix}finger_2_joint" type="prismatic">
@@ -81,5 +81,5 @@
       <child link="${tf_prefix}finger_2_link"/>
       <axis xyz="1 0 0"/>
-      <limit effort="130" lower="0" upper="0.025" velocity="0.15"/>
+      <limit effort="185" lower="0" upper="0.025" velocity="0.15"/>
       <mimic joint="${tf_prefix}finger_1_joint" multiplier="1" offset="0"/>
     </joint>
